Commit message: Updated inv kinematics + added testing file

File: src/inv_kinematics/scripts/CPMOVER6.urdf (robot description, URDF)
Before this commit: robot CPRMover6, 7 links, 6 joints
Joints:
- joint joint1: limit effort=100 velocity=30 -> lower=-2.27 upper=2.27 effort=100 velocity=30; type continuous -> revolute
- joint joint2: limit effort=100 velocity=30 -> lower=-0.87 upper=1.05 effort=100 velocity=30; type continuous -> revolute
- joint joint3: limit effort=100 velocity=30 -> lower=-1.92 upper=1.31 effort=100 velocity=30; type continuous -> revolute
- joint joint4: limit effort=100 velocity=30 -> lower=-2.44 upper=2.44 effort=100 velocity=30; type continuous -> revolute
- joint joint5: limit effort=100 velocity=30 -> lower=-1.22 upper=1.05 effort=100 velocity=40; type continuous -> revolute
- joint joint6: limit effort=100 velocity=30 -> lower=-2.09 upper=2.09 effort=100 velocity=100; type continuous -> revolute
