Commit message: Rename file paths

File: src/mover6_gripper/urdf/GreiferZF_2016.urdf (robot description, URDF)
Before this commit: robot GreiferZF_2016, 3 links, 2 joints
Links:
- link base_link: geometry collision mesh filename=package://mover6_gripper/meshes/base_link.STL; visual mesh filename=package://mover6_gripper/meshes/base_link.STL
- link gripper_a: geometry collision mesh filename=package://mover6_gripper/meshes/gripper_a.STL; visual mesh filename=package://mover6_gripper/meshes/gripper_a.STL
- link gripper_b: geometry collision mesh filename=package://mover6_gripper/meshes/gripper_b.STL; visual mesh filename=package://mover6_gripper/meshes/gripper_b.STL
