Commit message: updated gripper model

File: src/mover6_gripper/urdf/GreiferZF_2016.SLDASM.urdf (robot description, URDF)
Before this commit: robot GreiferZF_2016, 3 links, 2 joints
Links:
- link base_link: mass 0.0420250780697651 -> 0.0481254395674383
- link gripper_a: mass 0.00998043833114313 -> 0.009672
- link gripper_b: mass 0.00998043833114302 -> 0.009672
Joints:
- joint joint_a: axis 1 0 0 -> 0 0 0; origin xyz=-0.0105 0.00085663 -0.029246 rpy=-2.8041 0 1.5708 -> xyz=-0.0055607 -0.0041434 -0.04688 rpy=1.5708 -0.33752 3.1416
- joint joint_b: axis 1 0 0 -> 0 0 0; mimic joint=joint_a multiplier=1 offset=0 -> (none); origin xyz=0.0105 0 -0.029246 rpy=-2.8041 0 -1.5708 -> xyz=0.0055607 0.005 -0.04688 rpy=1.5708 -0.33752 0
