Commit message: Grouded robot

File: src/mover6_description/urdf/CPRMover6.urdf.xacro (robot description, xacro)
@@ -3,4 +3,10 @@
 <!-- URDF file for the Commonplace Robotics Mover4 robot arm -->
 <!-- Version 1.1 from Oct. 04th, 2016. -->
+  <!-- Used for fixing robot to Gazebo 'base_link' -->
+  <link name="world"/>
+  <joint name="fixed" type="fixed">
+    <parent link="world"/>
+    <child link="base_link"/>
+  </joint>
 <!-- Default Inertial -->
   <xacro:macro name="default_inertial" params="z_value mass">

Commit message: Updated urdf to use correct mesh Added transmission elements

File: src/mover6_description/urdf/CPRMover6.urdf.xacro (robot description, xacro)
@@ -29,5 +29,5 @@
       <origin xyz="0 0 0" rpy="0 0 0" />
       <geometry>
-          <mesh filename="package://cpr_robot/robots/CPRMover6/Joint0Coll.dae" scale="0.001 0.001 0.001"/>
+          <mesh filename="package://mover6_description/meshes/Joint0Coll.dae" scale="0.001 0.001 0.001"/>
         </geometry>
     </collision>
@@ -38,11 +38,11 @@
 	  <origin rpy="0 0 0" xyz="0 0 0"/>
       <geometry>
-          <mesh filename="package://cpr_robot/robots/CPRMover6/Joint1.dae"  scale="0.001 0.001 0.001"/>
-        </geometry>
-    </visual>
-    <collision>
-      <origin xyz="0 0 0" rpy="0 0 0" />
-      <geometry>
-          <mesh filename="package://cpr_robot/robots/CPRMover6/Joint1Coll.dae" scale="0.001 0.001 0.001"/>
+          <mesh filename="package://mover6_description/meshes/Joint1.dae"  scale="0.001 0.001 0.001"/>
+        </geometry>
+    </visual>
+    <collision>
+      <origin xyz="0 0 0" rpy="0 0 0" />
+      <geometry>
+          <mesh filename="package://mover6_description/meshes/Joint1Coll.dae" scale="0.001 0.001 0.001"/>
         </geometry>
     </collision>
@@ -53,11 +53,11 @@
 	  <origin rpy="0 0 0" xyz="0 0 0"/>
       <geometry>
-          <mesh filename="package://cpr_robot/robots/CPRMover6/Joint2.dae"  scale="0.001 0.001 0.001"/>
-        </geometry>
-    </visual>
-    <collision>
-      <origin xyz="0 0 0" rpy="0 0 0" />
-      <geometry>
-          <mesh filename="package://cpr_robot/robots/CPRMover6/Joint2Coll.dae" scale="0.001 0.001 0.001"/>
+          <mesh filename="package://mover6_description/meshes/Joint2.dae"  scale="0.001 0.001 0.001"/>
+        </geometry>
+    </visual>
+    <collision>
+      <origin xyz="0 0 0" rpy="0 0 0" />
+      <geometry>
+          <mesh filename="package://mover6_description/meshes/Joint2Coll.dae" scale="0.001 0.001 0.001"/>
         </geometry>
     </collision>
@@ -68,11 +68,11 @@
 	  <origin rpy="0 0 0" xyz="0 0 0"/>
       <geometry>
-          <mesh filename="package://cpr_robot/robots/CPRMover6/Joint3.dae"  scale="0.001 0.001 0.001"/>
-        </geometry>
-    </visual>
-    <collision>
-      <origin xyz="0 0 0" rpy="0 0 0" />
-      <geometry>
-          <mesh filename="package://cpr_robot/robots/CPRMover6/Joint3Coll.dae" scale="0.001 0.001 0.001"/>
+          <mesh filename="package://mover6_description/meshes/Joint3.dae"  scale="0.001 0.001 0.001"/>
+        </geometry>
+    </visual>
+    <collision>
+      <origin xyz="0 0 0" rpy="0 0 0" />
+      <geometry>
+          <mesh filename="package://mover6_description/meshes/Joint3Coll.dae" scale="0.001 0.001 0.001"/>
         </geometry>
     </collision>
@@ -83,11 +83,11 @@
 	  <origin rpy="0 0 0" xyz="0 0 0"/>
       <geometry>
-          <mesh filename="package://cpr_robot/robots/CPRMover6/Joint4.dae"  scale="0.001 0.001 0.001"/>
-        </geometry>
-    </visual>
-    <collision>
-      <origin xyz="0 0 0" rpy="0 0 0" />
-      <geometry>
-          <mesh filename="package://cpr_robot/robots/CPRMover6/Joint4Coll.dae" scale="0.001 0.001 0.001"/>
+          <mesh filename="package://mover6_description/meshes/Joint4.dae"  scale="0.001 0.001 0.001"/>
+        </geometry>
+    </visual>
+    <collision>
+      <origin xyz="0 0 0" rpy="0 0 0" />
+      <geometry>
+          <mesh filename="package://mover6_description/meshes/Joint4Coll.dae" scale="0.001 0.001 0.001"/>
         </geometry>
     </collision>
@@ -98,11 +98,11 @@
 	  <origin rpy="0 0 0" xyz="0 0 0"/>
       <geometry>
-          <mesh filename="package://cpr_robot/robots/CPRMover6/Joint5.dae"  scale="0.001 0.001 0.001"/>
-        </geometry>
-    </visual>
-    <collision>
-      <origin xyz="0 0 0" rpy="0 0 0" />
-      <geometry>
-          <mesh filename="package://cpr_robot/robots/CPRMover6/Joint5Coll.dae" scale="0.001 0.001 0.001"/>
+          <mesh filename="package://mover6_description/meshes/Joint5.dae"  scale="0.001 0.001 0.001"/>
+        </geometry>
+    </visual>
+    <collision>
+      <origin xyz="0 0 0" rpy="0 0 0" />
+      <geometry>
+          <mesh filename="package://mover6_description/meshes/Joint5Coll.dae" scale="0.001 0.001 0.001"/>
         </geometry>
     </collision>
@@ -113,11 +113,11 @@
 	  <origin rpy="0 0 0" xyz="0 0 0"/>
       <geometry>
-          <mesh filename="package://cpr_robot/robots/CPRMover6/Joint6.dae"  scale="0.001 0.001 0.001"/>
-        </geometry>
-    </visual>
-    <collision>
-      <origin xyz="0 0 0" rpy="0 0 0" />
-      <geometry>
-          <mesh filename="package://cpr_robot/robots/CPRMover6/Joint6Coll.dae" scale="0.001 0.001 0.001"/>
+          <mesh filename="package://mover6_description/meshes/Joint6.dae"  scale="0.001 0.001 0.001"/>
+        </geometry>
+    </visual>
+    <collision>
+      <origin xyz="0 0 0" rpy="0 0 0" />
+      <geometry>
+          <mesh filename="package://mover6_description/meshes/Joint6Coll.dae" scale="0.001 0.001 0.001"/>
         </geometry>
     </collision>
@@ -172,3 +172,63 @@
     <joint_properties damping="0.0" friction="0.0"/>
   </joint>
+  <transmission name="tran1">
+<type>transmission_interface/SimpleTransmission</type>
+<joint name="joint1">
+    <hardwareInterface>EffortJointInterface</hardwareInterface>
+</joint>
+<actuator name="motor1">
+    <hardwareInterface>EffortJointInterface</hardwareInterface>
+    <mechanicalReduction>1</mechanicalReduction>
+</actuator>
+</transmission>
+<transmission name="tran2">
+<type>transmission_interface/SimpleTransmission</type>
+<joint name="joint2">
+    <hardwareInterface>EffortJointInterface</hardwareInterface>
+</joint>
+<actuator name="motor2">
+    <hardwareInterface>EffortJointInterface</hardwareInterface>
+    <mechanicalReduction>1</mechanicalReduction>
+</actuator>
+</transmission>
+<transmission name="tran3">
+<type>transmission_interface/SimpleTransmission</type>
+<joint name="joint3">
+    <hardwareInterface>EffortJointInterface</hardwareInterface>
+</joint>
+<actuator name="motor3">
+    <hardwareInterface>EffortJointInterface</hardwareInterface>
+    <mechanicalReduction>1</mechanicalReduction>
+</actuator>
+</transmission>
+<transmission name="tran4">
+<type>transmission_interface/SimpleTransmission</type>
+<joint name="joint4">
+    <hardwareInterface>EffortJointInterface</hardwareInterface>
+</joint>
+<actuator name="motor4">
+    <hardwareInterface>EffortJointInterface</hardwareInterface>
+    <mechanicalReduction>1</mechanicalReduction>
+</actuator>
+</transmission>
+<transmission name="tran5">
+<type>transmission_interface/SimpleTransmission</type>
+<joint name="joint5">
+    <hardwareInterface>EffortJointInterface</hardwareInterface>
+</joint>
+<actuator name="motor5">
+    <hardwareInterface>EffortJointInterface</hardwareInterface>
+    <mechanicalReduction>1</mechanicalReduction>
+</actuator>
+</transmission>
+<transmission name="tran6">
+<type>transmission_interface/SimpleTransmission</type>
+<joint name="joint6">
+    <hardwareInterface>EffortJointInterface</hardwareInterface>
+</joint>
+<actuator name="motor6">
+    <hardwareInterface>EffortJointInterface</hardwareInterface>
+    <mechanicalReduction>1</mechanicalReduction>
+</actuator>
+</transmission>
 </robot>

Commit message: Tidy urdf

File: src/mover6_description/urdf/CPRMover6.urdf.xacro (robot description, xacro)
@@ -1,234 +1,235 @@
 <?xml version="1.0"?>
-<robot xmlns:xacro="http://ros.org/wiki/xacro" name="CPRMover6">
-<!-- URDF file for the Commonplace Robotics Mover4 robot arm -->
-<!-- Version 1.1 from Oct. 04th, 2016. -->
-  <!-- Used for fixing robot to Gazebo 'base_link' -->
-  <link name="world"/>
-  <joint name="fixed" type="fixed">
-    <parent link="world"/>
-    <child link="base_link"/>
-  </joint>
-<!-- Default Inertial -->
-  <xacro:macro name="default_inertial" params="z_value mass">
-    <inertial>
-      <origin xyz="0 0 ${z_value}" rpy="0 0 0"/>
-      <mass value="${mass}" />
-      <inertia ixx="1.0" ixy="0.0" ixz="0.0"
+<robot
+	xmlns:xacro="http://ros.org/wiki/xacro" name="CPRMover6">
+	<!-- URDF file for the Commonplace Robotics Mover4 robot arm -->
+	<!-- Version 1.1 from Oct. 04th, 2016. -->
+	<!-- Used for fixing robot to Gazebo 'base_link' -->
+	<link name="world"/>
+	<joint name="fixed" type="fixed">
+		<parent link="world"/>
+		<child link="base_link"/>
+	</joint>
+	<!-- Default Inertial -->
+	<xacro:macro name="default_inertial" params="z_value mass">
+		<inertial>
+			<origin xyz="0 0 ${z_value}" rpy="0 0 0"/>
+			<mass value="${mass}" />
+			<inertia ixx="1.0" ixy="0.0" ixz="0.0"
                iyy="1.0" iyz="0.0"
                izz="1.0" />
-      </inertial>
-  </xacro:macro>
-  <link name="base_link">
-    <visual>
-	  <origin rpy="0 0 0" xyz="0 0 0"/>
-      <geometry>
-          <mesh filename="package://mover6_description/meshes/Joint0.stl"  scale="0.001 0.001 0.001"/>
-        </geometry>
-    </visual>
-    <collision>
-      <origin xyz="0 0 0" rpy="0 0 0" />
-      <geometry>
-          <mesh filename="package://mover6_description/meshes/Joint0Coll.dae" scale="0.001 0.001 0.001"/>
-        </geometry>
-    </collision>
-    <xacro:default_inertial z_value="0" mass="1"/>
-  </link>
-  <link name="link1">
-    <visual>
-	  <origin rpy="0 0 0" xyz="0 0 0"/>
-      <geometry>
-          <mesh filename="package://mover6_description/meshes/Joint1.dae"  scale="0.001 0.001 0.001"/>
-        </geometry>
-    </visual>
-    <collision>
-      <origin xyz="0 0 0" rpy="0 0 0" />
-      <geometry>
-          <mesh filename="package://mover6_description/meshes/Joint1Coll.dae" scale="0.001 0.001 0.001"/>
-        </geometry>
-    </collision>
-    <xacro:default_inertial z_value="0" mass="1"/>
-  </link>
-  <link name="link2">
-    <visual>
-	  <origin rpy="0 0 0" xyz="0 0 0"/>
-      <geometry>
-          <mesh filename="package://mover6_description/meshes/Joint2.dae"  scale="0.001 0.001 0.001"/>
-        </geometry>
-    </visual>
-    <collision>
-      <origin xyz="0 0 0" rpy="0 0 0" />
-      <geometry>
-          <mesh filename="package://mover6_description/meshes/Joint2Coll.dae" scale="0.001 0.001 0.001"/>
-        </geometry>
-    </collision>
-    <xacro:default_inertial z_value="0" mass="1"/>
-  </link>
-  <link name="link3">
-    <visual>
-	  <origin rpy="0 0 0" xyz="0 0 0"/>
-      <geometry>
-          <mesh filename="package://mover6_description/meshes/Joint3.dae"  scale="0.001 0.001 0.001"/>
-        </geometry>
-    </visual>
-    <collision>
-      <origin xyz="0 0 0" rpy="0 0 0" />
-      <geometry>
-          <mesh filename="package://mover6_description/meshes/Joint3Coll.dae" scale="0.001 0.001 0.001"/>
-        </geometry>
-    </collision>
-    <xacro:default_inertial z_value="0" mass="1"/>
-  </link>
-  <link name="link4">
-    <visual>
-	  <origin rpy="0 0 0" xyz="0 0 0"/>
-      <geometry>
-          <mesh filename="package://mover6_description/meshes/Joint4.dae"  scale="0.001 0.001 0.001"/>
-        </geometry>
-    </visual>
-    <collision>
-      <origin xyz="0 0 0" rpy="0 0 0" />
-      <geometry>
-          <mesh filename="package://mover6_description/meshes/Joint4Coll.dae" scale="0.001 0.001 0.001"/>
-        </geometry>
-    </collision>
-    <xacro:default_inertial z_value="0" mass="1"/>
-  </link>
-  <link name="link5">
-    <visual>
-	  <origin rpy="0 0 0" xyz="0 0 0"/>
-      <geometry>
-          <mesh filename="package://mover6_description/meshes/Joint5.dae"  scale="0.001 0.001 0.001"/>
-        </geometry>
-    </visual>
-    <collision>
-      <origin xyz="0 0 0" rpy="0 0 0" />
-      <geometry>
-          <mesh filename="package://mover6_description/meshes/Joint5Coll.dae" scale="0.001 0.001 0.001"/>
-        </geometry>
-    </collision>
-    <xacro:default_inertial z_value="0" mass="1"/>
-  </link>
-  <link name="link6">
-    <visual>
-	  <origin rpy="0 0 0" xyz="0 0 0"/>
-      <geometry>
-          <mesh filename="package://mover6_description/meshes/Joint6.dae"  scale="0.001 0.001 0.001"/>
-        </geometry>
-    </visual>
-    <collision>
-      <origin xyz="0 0 0" rpy="0 0 0" />
-      <geometry>
-          <mesh filename="package://mover6_description/meshes/Joint6Coll.dae" scale="0.001 0.001 0.001"/>
-        </geometry>
-    </collision>
-    <xacro:default_inertial z_value="0" mass="1"/>
-  </link>
-  <joint name="joint1" type="continuous">
-    <axis xyz="0 0 -1"/>
-    <parent link="base_link"/>
-    <child link="link1"/>
-    <origin rpy="0 0 0" xyz="0 0 0.130"/>
-    <limit effort="100" velocity="30"/>
-    <joint_properties damping="0.0" friction="0.0"/>
-  </joint>
-  <joint name="joint2" type="continuous">
-    <axis xyz="0 1 0"/>
-    <parent link="link1"/>
-    <child link="link2"/>
-    <origin rpy="0 0 0" xyz="0 0 0.0625"/>
-    <limit effort="100" velocity="30"/>
-    <joint_properties damping="0.0" friction="0.0"/>
-  </joint>
- <joint name="joint3" type="continuous">
-    <axis xyz="0 1 0"/>
-    <parent link="link2"/>
-    <child link="link3"/>
-    <origin rpy="0 1.57079632679 0" xyz="0 0 0.190"/>
-    <limit effort="100" velocity="30"/>
-    <joint_properties damping="0.0" friction="0.0"/>
-  </joint>
- <joint name="joint4" type="continuous">
-    <axis xyz="0 0 1"/>
-    <parent link="link3"/>
-    <child link="link4"/>
-    <origin rpy="0 0 0" xyz="-0.06 0 0"/>
-    <limit effort="100" velocity="30"/>
-    <joint_properties damping="0.0" friction="0.0"/>
-  </joint>
- <joint name="joint5" type="continuous">
-    <axis xyz="0 1 0"/>
-    <parent link="link4"/>
-    <child link="link5"/>
-    <origin rpy="0 0 0" xyz="0 0 0.290"/>
-    <limit effort="100" velocity="30"/>
-    <joint_properties damping="0.0" friction="0.0"/>
-  </joint>
- <joint name="joint6" type="continuous">
-    <axis xyz="0 0 1"/>
-    <parent link="link5"/>
-    <child link="link6"/>
-    <origin rpy="0 0 0" xyz="0 0 0.055"/>
-    <limit effort="100" velocity="30"/>
-    <joint_properties damping="0.0" friction="0.0"/>
-  </joint>
-  <transmission name="tran1">
-<type>transmission_interface/SimpleTransmission</type>
-<joint name="joint1">
-    <hardwareInterface>EffortJointInterface</hardwareInterface>
-</joint>
-<actuator name="motor1">
-    <hardwareInterface>EffortJointInterface</hardwareInterface>
-    <mechanicalReduction>1</mechanicalReduction>
-</actuator>
-</transmission>
-<transmission name="tran2">
-<type>transmission_interface/SimpleTransmission</type>
-<joint name="joint2">
-    <hardwareInterface>EffortJointInterface</hardwareInterface>
-</joint>
-<actuator name="motor2">
-    <hardwareInterface>EffortJointInterface</hardwareInterface>
-    <mechanicalReduction>1</mechanicalReduction>
-</actuator>
-</transmission>
-<transmission name="tran3">
-<type>transmission_interface/SimpleTransmission</type>
-<joint name="joint3">
-    <hardwareInterface>EffortJointInterface</hardwareInterface>
-</joint>
-<actuator name="motor3">
-    <hardwareInterface>EffortJointInterface</hardwareInterface>
-    <mechanicalReduction>1</mechanicalReduction>
-</actuator>
-</transmission>
-<transmission name="tran4">
-<type>transmission_interface/SimpleTransmission</type>
-<joint name="joint4">
-    <hardwareInterface>EffortJointInterface</hardwareInterface>
-</joint>
-<actuator name="motor4">
-    <hardwareInterface>EffortJointInterface</hardwareInterface>
-    <mechanicalReduction>1</mechanicalReduction>
-</actuator>
-</transmission>
-<transmission name="tran5">
-<type>transmission_interface/SimpleTransmission</type>
-<joint name="joint5">
-    <hardwareInterface>EffortJointInterface</hardwareInterface>
-</joint>
-<actuator name="motor5">
-    <hardwareInterface>EffortJointInterface</hardwareInterface>
-    <mechanicalReduction>1</mechanicalReduction>
-</actuator>
-</transmission>
-<transmission name="tran6">
-<type>transmission_interface/SimpleTransmission</type>
-<joint name="joint6">
-    <hardwareInterface>EffortJointInterface</hardwareInterface>
-</joint>
-<actuator name="motor6">
-    <hardwareInterface>EffortJointInterface</hardwareInterface>
-    <mechanicalReduction>1</mechanicalReduction>
-</actuator>
-</transmission>
+		</inertial>
+	</xacro:macro>
+	<link name="base_link">
+		<visual>
+			<origin rpy="0 0 0" xyz="0 0 0"/>
+			<geometry>
+				<mesh filename="package://mover6_description/meshes/Joint0.stl"  scale="0.001 0.001 0.001"/>
+			</geometry>
+		</visual>
+		<collision>
+			<origin xyz="0 0 0" rpy="0 0 0" />
+			<geometry>
+				<mesh filename="package://mover6_description/meshes/Joint0Coll.dae" scale="0.001 0.001 0.001"/>
+			</geometry>
+		</collision>
+		<xacro:default_inertial z_value="0" mass="1"/>
+	</link>
+	<link name="link1">
+		<visual>
+			<origin rpy="0 0 0" xyz="0 0 0"/>
+			<geometry>
+				<mesh filename="package://mover6_description/meshes/Joint1.dae"  scale="0.001 0.001 0.001"/>
+			</geometry>
+		</visual>
+		<collision>
+			<origin xyz="0 0 0" rpy="0 0 0" />
+			<geometry>
+				<mesh filename="package://mover6_description/meshes/Joint1Coll.dae" scale="0.001 0.001 0.001"/>
+			</geometry>
+		</collision>
+		<xacro:default_inertial z_value="0" mass="1"/>
+	</link>
+	<link name="link2">
+		<visual>
+			<origin rpy="0 0 0" xyz="0 0 0"/>
+			<geometry>
+				<mesh filename="package://mover6_description/meshes/Joint2.dae"  scale="0.001 0.001 0.001"/>
+			</geometry>
+		</visual>
+		<collision>
+			<origin xyz="0 0 0" rpy="0 0 0" />
+			<geometry>
+				<mesh filename="package://mover6_description/meshes/Joint2Coll.dae" scale="0.001 0.001 0.001"/>
+			</geometry>
+		</collision>
+		<xacro:default_inertial z_value="0" mass="1"/>
+	</link>
+	<link name="link3">
+		<visual>
+			<origin rpy="0 0 0" xyz="0 0 0"/>
+			<geometry>
+				<mesh filename="package://mover6_description/meshes/Joint3.dae"  scale="0.001 0.001 0.001"/>
+			</geometry>
+		</visual>
+		<collision>
+			<origin xyz="0 0 0" rpy="0 0 0" />
+			<geometry>
+				<mesh filename="package://mover6_description/meshes/Joint3Coll.dae" scale="0.001 0.001 0.001"/>
+			</geometry>
+		</collision>
+		<xacro:default_inertial z_value="0" mass="1"/>
+	</link>
+	<link name="link4">
+		<visual>
+			<origin rpy="0 0 0" xyz="0 0 0"/>
+			<geometry>
+				<mesh filename="package://mover6_description/meshes/Joint4.dae"  scale="0.001 0.001 0.001"/>
+			</geometry>
+		</visual>
+		<collision>
+			<origin xyz="0 0 0" rpy="0 0 0" />
+			<geometry>
+				<mesh filename="package://mover6_description/meshes/Joint4Coll.dae" scale="0.001 0.001 0.001"/>
+			</geometry>
+		</collision>
+		<xacro:default_inertial z_value="0" mass="1"/>
+	</link>
+	<link name="link5">
+		<visual>
+			<origin rpy="0 0 0" xyz="0 0 0"/>
+			<geometry>
+				<mesh filename="package://mover6_description/meshes/Joint5.dae"  scale="0.001 0.001 0.001"/>
+			</geometry>
+		</visual>
+		<collision>
+			<origin xyz="0 0 0" rpy="0 0 0" />
+			<geometry>
+				<mesh filename="package://mover6_description/meshes/Joint5Coll.dae" scale="0.001 0.001 0.001"/>
+			</geometry>
+		</collision>
+		<xacro:default_inertial z_value="0" mass="1"/>
+	</link>
+	<link name="link6">
+		<visual>
+			<origin rpy="0 0 0" xyz="0 0 0"/>
+			<geometry>
+				<mesh filename="package://mover6_description/meshes/Joint6.dae"  scale="0.001 0.001 0.001"/>
+			</geometry>
+		</visual>
+		<collision>
+			<origin xyz="0 0 0" rpy="0 0 0" />
+			<geometry>
+				<mesh filename="package://mover6_description/meshes/Joint6Coll.dae" scale="0.001 0.001 0.001"/>
+			</geometry>
+		</collision>
+		<xacro:default_inertial z_value="0" mass="1"/>
+	</link>
+	<joint name="joint1" type="continuous">
+		<axis xyz="0 0 -1"/>
+		<parent link="base_link"/>
+		<child link="link1"/>
+		<origin rpy="0 0 0" xyz="0 0 0.130"/>
+		<limit effort="100" velocity="30"/>
+		<joint_properties damping="0.0" friction="0.0"/>
+	</joint>
+	<joint name="joint2" type="continuous">
+		<axis xyz="0 1 0"/>
+		<parent link="link1"/>
+		<child link="link2"/>
+		<origin rpy="0 0 0" xyz="0 0 0.0625"/>
+		<limit effort="100" velocity="30"/>
+		<joint_properties damping="0.0" friction="0.0"/>
+	</joint>
+	<joint name="joint3" type="continuous">
+		<axis xyz="0 1 0"/>
+		<parent link="link2"/>
+		<child link="link3"/>
+		<origin rpy="0 1.57079632679 0" xyz="0 0 0.190"/>
+		<limit effort="100" velocity="30"/>
+		<joint_properties damping="0.0" friction="0.0"/>
+	</joint>
+	<joint name="joint4" type="continuous">
+		<axis xyz="0 0 1"/>
+		<parent link="link3"/>
+		<child link="link4"/>
+		<origin rpy="0 0 0" xyz="-0.06 0 0"/>
+		<limit effort="100" velocity="30"/>
+		<joint_properties damping="0.0" friction="0.0"/>
+	</joint>
+	<joint name="joint5" type="continuous">
+		<axis xyz="0 1 0"/>
+		<parent link="link4"/>
+		<child link="link5"/>
+		<origin rpy="0 0 0" xyz="0 0 0.290"/>
+		<limit effort="100" velocity="30"/>
+		<joint_properties damping="0.0" friction="0.0"/>
+	</joint>
+	<joint name="joint6" type="continuous">
+		<axis xyz="0 0 1"/>
+		<parent link="link5"/>
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