Commit message: Initial arm parameter tuning

File: src/mover6_description/urdf/CPRMover6.urdf.xacro (robot description, xacro)
@@ -33,5 +33,5 @@
 			</geometry>
 		</collision>
-		<xacro:default_inertial z_value="0" mass="1"/>
+		<xacro:default_inertial z_value="0" mass="1.5"/>
 	</link>
 	<link name="link1">
@@ -48,5 +48,5 @@
 			</geometry>
 		</collision>
-		<xacro:default_inertial z_value="0" mass="1"/>
+		<xacro:default_inertial z_value="0" mass="0.5"/>
 	</link>
 	<link name="link2">
@@ -63,5 +63,5 @@
 			</geometry>
 		</collision>
-		<xacro:default_inertial z_value="0" mass="1"/>
+		<xacro:default_inertial z_value="0" mass="0.5"/>
 	</link>
 	<link name="link3">
@@ -78,5 +78,5 @@
 			</geometry>
 		</collision>
-		<xacro:default_inertial z_value="0" mass="1"/>
+		<xacro:default_inertial z_value="0" mass="0.5"/>
 	</link>
 	<link name="link4">
@@ -93,5 +93,5 @@
 			</geometry>
 		</collision>
-		<xacro:default_inertial z_value="0" mass="1"/>
+		<xacro:default_inertial z_value="0" mass="0.2"/>
 	</link>
 	<link name="link5">
@@ -108,5 +108,5 @@
 			</geometry>
 		</collision>
-		<xacro:default_inertial z_value="0" mass="1"/>
+		<xacro:default_inertial z_value="0" mass="0.2"/>
 	</link>
 	<link name="link6">
@@ -123,53 +123,53 @@
 			</geometry>
 		</collision>
-		<xacro:default_inertial z_value="0" mass="1"/>
-	</link>
-	<joint name="joint1" type="continuous">
+		<xacro:default_inertial z_value="0" mass="0.1"/>
+	</link>
+	<joint name="joint1" type="revolute">
 		<axis xyz="0 0 -1"/>
 		<parent link="base_link"/>
 		<child link="link1"/>
 		<origin rpy="0 0 0" xyz="0 0 0.130"/>
-		<limit effort="100" velocity="30"/>
-		<joint_properties damping="0.0" friction="0.0"/>
-	</joint>
-	<joint name="joint2" type="continuous">
+		<limit lower="-2.27" upper="2.27" effort="100" velocity="30"/>
+		<joint_properties damping="1.0" friction="10.0"/>
+	</joint>
+	<joint name="joint2" type="revolute">
 		<axis xyz="0 1 0"/>
 		<parent link="link1"/>
 		<child link="link2"/>
 		<origin rpy="0 0 0" xyz="0 0 0.0625"/>
-		<limit effort="100" velocity="30"/>
-		<joint_properties damping="0.0" friction="0.0"/>
-	</joint>
-	<joint name="joint3" type="continuous">
+		<limit lower="-0.87" upper="1.05" effort="100" velocity="30"/>
+		<joint_properties damping="1.0" friction="10.0"/>
+	</joint>
+	<joint name="joint3" type="revolute">
 		<axis xyz="0 1 0"/>
 		<parent link="link2"/>
 		<child link="link3"/>
 		<origin rpy="0 1.57079632679 0" xyz="0 0 0.190"/>
-		<limit effort="100" velocity="30"/>
-		<joint_properties damping="0.0" friction="0.0"/>
-	</joint>
-	<joint name="joint4" type="continuous">
+		<limit lower="-1.92" upper="1.31" effort="100" velocity="30"/>
+		<joint_properties damping="1.0" friction="10.0"/>
+	</joint>
+	<joint name="joint4" type="revolute">
 		<axis xyz="0 0 1"/>
 		<parent link="link3"/>
 		<child link="link4"/>
 		<origin rpy="0 0 0" xyz="-0.06 0 0"/>
-		<limit effort="100" velocity="30"/>
-		<joint_properties damping="0.0" friction="0.0"/>
-	</joint>
-	<joint name="joint5" type="continuous">
+		<limit lower="-2.44" upper="2.44" effort="100" velocity="30"/>
+		<joint_properties damping="1.0" friction="10.0"/>
+	</joint>
+	<joint name="joint5" type="revolute">
 		<axis xyz="0 1 0"/>
 		<parent link="link4"/>
 		<child link="link5"/>
 		<origin rpy="0 0 0" xyz="0 0 0.290"/>
-		<limit effort="100" velocity="30"/>
-		<joint_properties damping="0.0" friction="0.0"/>
-	</joint>
-	<joint name="joint6" type="continuous">
+		<limit lower="-1.22" upper="1.05" effort="100" velocity="40"/>
+		<joint_properties damping="1.0" friction="1.0"/>
+	</joint>
+	<joint name="joint6" type="revolute">
 		<axis xyz="0 0 1"/>
 		<parent link="link5"/>
 		<child link="link6"/>
 		<origin rpy="0 0 0" xyz="0 0 0.055"/>
-		<limit effort="100" velocity="30"/>
-		<joint_properties damping="0.0" friction="0.0"/>
+		<limit lower="-2.09" upper="2.09" effort="100" velocity="100"/>
+		<joint_properties damping="1.0" friction="1.0"/>
 	</joint>
 	<transmission name="tran1">

Commit message: Add ROS-Control functions (#1)
* Tidy urdf

* Setup ros control mostly

* updated mover6 gazebo launch file names

* Updated urdf to remove error msg

* Setup controller

* Updated talker to run all joints

* Add python run script

* Initial arm parameter tuning

* Updated talker to randomly move all joints

* Update sim joint test

File: src/mover6_description/urdf/CPRMover6.urdf.xacro (robot description, xacro)
@@ -1,234 +1,240 @@
 <?xml version="1.0"?>
-<robot xmlns:xacro="http://ros.org/wiki/xacro" name="CPRMover6">
-<!-- URDF file for the Commonplace Robotics Mover4 robot arm -->
-<!-- Version 1.1 from Oct. 04th, 2016. -->
-  <!-- Used for fixing robot to Gazebo 'base_link' -->
-  <link name="world"/>
-  <joint name="fixed" type="fixed">
-    <parent link="world"/>
-    <child link="base_link"/>
-  </joint>
-<!-- Default Inertial -->
-  <xacro:macro name="default_inertial" params="z_value mass">
-    <inertial>
-      <origin xyz="0 0 ${z_value}" rpy="0 0 0"/>
-      <mass value="${mass}" />
-      <inertia ixx="1.0" ixy="0.0" ixz="0.0"
+<robot
+	xmlns:xacro="http://ros.org/wiki/xacro" name="CPRMover6">
+	<!-- URDF file for the Commonplace Robotics Mover4 robot arm -->
+	<!-- Version 1.1 from Oct. 04th, 2016. -->
+	<!-- Used for fixing robot to Gazebo 'base_link' -->
+	<link name="world"/>
+	<joint name="fixed" type="fixed">
+		<parent link="world"/>
+		<child link="base_link"/>
+	</joint>
+	<!-- Default Inertial -->
+	<xacro:macro name="default_inertial" params="z_value mass">
+		<inertial>
+			<origin xyz="0 0 ${z_value}" rpy="0 0 0"/>
+			<mass value="${mass}" />
+			<inertia ixx="1.0" ixy="0.0" ixz="0.0"
                iyy="1.0" iyz="0.0"
                izz="1.0" />
-      </inertial>
-  </xacro:macro>
-  <link name="base_link">
-    <visual>
-	  <origin rpy="0 0 0" xyz="0 0 0"/>
-      <geometry>
-          <mesh filename="package://mover6_description/meshes/Joint0.stl"  scale="0.001 0.001 0.001"/>
-        </geometry>
-    </visual>
-    <collision>
-      <origin xyz="0 0 0" rpy="0 0 0" />
-      <geometry>
-          <mesh filename="package://mover6_description/meshes/Joint0Coll.dae" scale="0.001 0.001 0.001"/>
-        </geometry>
-    </collision>
-    <xacro:default_inertial z_value="0" mass="1"/>
-  </link>
-  <link name="link1">
-    <visual>
-	  <origin rpy="0 0 0" xyz="0 0 0"/>
-      <geometry>
-          <mesh filename="package://mover6_description/meshes/Joint1.dae"  scale="0.001 0.001 0.001"/>
-        </geometry>
-    </visual>
-    <collision>
-      <origin xyz="0 0 0" rpy="0 0 0" />
-      <geometry>
-          <mesh filename="package://mover6_description/meshes/Joint1Coll.dae" scale="0.001 0.001 0.001"/>
-        </geometry>
-    </collision>
-    <xacro:default_inertial z_value="0" mass="1"/>
-  </link>
-  <link name="link2">
-    <visual>
-	  <origin rpy="0 0 0" xyz="0 0 0"/>
-      <geometry>
-          <mesh filename="package://mover6_description/meshes/Joint2.dae"  scale="0.001 0.001 0.001"/>
-        </geometry>
-    </visual>
-    <collision>
-      <origin xyz="0 0 0" rpy="0 0 0" />
-      <geometry>
-          <mesh filename="package://mover6_description/meshes/Joint2Coll.dae" scale="0.001 0.001 0.001"/>
-        </geometry>
-    </collision>
-    <xacro:default_inertial z_value="0" mass="1"/>
-  </link>
-  <link name="link3">
-    <visual>
-	  <origin rpy="0 0 0" xyz="0 0 0"/>
-      <geometry>
-          <mesh filename="package://mover6_description/meshes/Joint3.dae"  scale="0.001 0.001 0.001"/>
-        </geometry>
-    </visual>
-    <collision>
-      <origin xyz="0 0 0" rpy="0 0 0" />
-      <geometry>
-          <mesh filename="package://mover6_description/meshes/Joint3Coll.dae" scale="0.001 0.001 0.001"/>
-        </geometry>
-    </collision>
-    <xacro:default_inertial z_value="0" mass="1"/>
-  </link>
-  <link name="link4">
-    <visual>
-	  <origin rpy="0 0 0" xyz="0 0 0"/>
-      <geometry>
-          <mesh filename="package://mover6_description/meshes/Joint4.dae"  scale="0.001 0.001 0.001"/>
-        </geometry>
-    </visual>
-    <collision>
-      <origin xyz="0 0 0" rpy="0 0 0" />
-      <geometry>
-          <mesh filename="package://mover6_description/meshes/Joint4Coll.dae" scale="0.001 0.001 0.001"/>
-        </geometry>
-    </collision>
-    <xacro:default_inertial z_value="0" mass="1"/>
-  </link>
-  <link name="link5">
-    <visual>
-	  <origin rpy="0 0 0" xyz="0 0 0"/>
-      <geometry>
-          <mesh filename="package://mover6_description/meshes/Joint5.dae"  scale="0.001 0.001 0.001"/>
-        </geometry>
-    </visual>
-    <collision>
-      <origin xyz="0 0 0" rpy="0 0 0" />
-      <geometry>
-          <mesh filename="package://mover6_description/meshes/Joint5Coll.dae" scale="0.001 0.001 0.001"/>
-        </geometry>
-    </collision>
-    <xacro:default_inertial z_value="0" mass="1"/>
-  </link>
-  <link name="link6">
-    <visual>
-	  <origin rpy="0 0 0" xyz="0 0 0"/>
-      <geometry>
-          <mesh filename="package://mover6_description/meshes/Joint6.dae"  scale="0.001 0.001 0.001"/>
-        </geometry>
-    </visual>
-    <collision>
-      <origin xyz="0 0 0" rpy="0 0 0" />
-      <geometry>
-          <mesh filename="package://mover6_description/meshes/Joint6Coll.dae" scale="0.001 0.001 0.001"/>
-        </geometry>
-    </collision>
-    <xacro:default_inertial z_value="0" mass="1"/>
-  </link>
-  <joint name="joint1" type="continuous">
-    <axis xyz="0 0 -1"/>
-    <parent link="base_link"/>
-    <child link="link1"/>
-    <origin rpy="0 0 0" xyz="0 0 0.130"/>
-    <limit effort="100" velocity="30"/>
-    <joint_properties damping="0.0" friction="0.0"/>
-  </joint>
-  <joint name="joint2" type="continuous">
-    <axis xyz="0 1 0"/>
-    <parent link="link1"/>
-    <child link="link2"/>
-    <origin rpy="0 0 0" xyz="0 0 0.0625"/>
-    <limit effort="100" velocity="30"/>
-    <joint_properties damping="0.0" friction="0.0"/>
-  </joint>
- <joint name="joint3" type="continuous">
-    <axis xyz="0 1 0"/>
-    <parent link="link2"/>
-    <child link="link3"/>
-    <origin rpy="0 1.57079632679 0" xyz="0 0 0.190"/>
-    <limit effort="100" velocity="30"/>
-    <joint_properties damping="0.0" friction="0.0"/>
-  </joint>
- <joint name="joint4" type="continuous">
-    <axis xyz="0 0 1"/>
-    <parent link="link3"/>
-    <child link="link4"/>
-    <origin rpy="0 0 0" xyz="-0.06 0 0"/>
-    <limit effort="100" velocity="30"/>
-    <joint_properties damping="0.0" friction="0.0"/>
-  </joint>
- <joint name="joint5" type="continuous">
-    <axis xyz="0 1 0"/>
-    <parent link="link4"/>
-    <child link="link5"/>
-    <origin rpy="0 0 0" xyz="0 0 0.290"/>
-    <limit effort="100" velocity="30"/>
-    <joint_properties damping="0.0" friction="0.0"/>
-  </joint>
- <joint name="joint6" type="continuous">
-    <axis xyz="0 0 1"/>
-    <parent link="link5"/>
-    <child link="link6"/>
-    <origin rpy="0 0 0" xyz="0 0 0.055"/>
-    <limit effort="100" velocity="30"/>
-    <joint_properties damping="0.0" friction="0.0"/>
-  </joint>
-  <transmission name="tran1">
-<type>transmission_interface/SimpleTransmission</type>
-<joint name="joint1">
-    <hardwareInterface>EffortJointInterface</hardwareInterface>
-</joint>
-<actuator name="motor1">
-    <hardwareInterface>EffortJointInterface</hardwareInterface>
-    <mechanicalReduction>1</mechanicalReduction>
-</actuator>
-</transmission>
-<transmission name="tran2">
-<type>transmission_interface/SimpleTransmission</type>
-<joint name="joint2">
-    <hardwareInterface>EffortJointInterface</hardwareInterface>
-</joint>
-<actuator name="motor2">
-    <hardwareInterface>EffortJointInterface</hardwareInterface>
-    <mechanicalReduction>1</mechanicalReduction>
-</actuator>
-</transmission>
-<transmission name="tran3">
-<type>transmission_interface/SimpleTransmission</type>
-<joint name="joint3">
-    <hardwareInterface>EffortJointInterface</hardwareInterface>
-</joint>
-<actuator name="motor3">
-    <hardwareInterface>EffortJointInterface</hardwareInterface>
-    <mechanicalReduction>1</mechanicalReduction>
-</actuator>
-</transmission>
-<transmission name="tran4">
-<type>transmission_interface/SimpleTransmission</type>
-<joint name="joint4">
-    <hardwareInterface>EffortJointInterface</hardwareInterface>
-</joint>
-<actuator name="motor4">
-    <hardwareInterface>EffortJointInterface</hardwareInterface>
-    <mechanicalReduction>1</mechanicalReduction>
-</actuator>
-</transmission>
-<transmission name="tran5">
-<type>transmission_interface/SimpleTransmission</type>
-<joint name="joint5">
-    <hardwareInterface>EffortJointInterface</hardwareInterface>
-</joint>
-<actuator name="motor5">
-    <hardwareInterface>EffortJointInterface</hardwareInterface>
-    <mechanicalReduction>1</mechanicalReduction>
-</actuator>
-</transmission>
-<transmission name="tran6">
-<type>transmission_interface/SimpleTransmission</type>
-<joint name="joint6">
-    <hardwareInterface>EffortJointInterface</hardwareInterface>
-</joint>
-<actuator name="motor6">
-    <hardwareInterface>EffortJointInterface</hardwareInterface>
-    <mechanicalReduction>1</mechanicalReduction>
-</actuator>
-</transmission>
+		</inertial>
+	</xacro:macro>
+	<link name="base_link">
+		<visual>
+			<origin rpy="0 0 0" xyz="0 0 0"/>
+			<geometry>
+				<mesh filename="package://mover6_description/meshes/Joint0.stl"  scale="0.001 0.001 0.001"/>
+			</geometry>
+		</visual>
+		<collision>
+			<origin xyz="0 0 0" rpy="0 0 0" />
+			<geometry>
+				<mesh filename="package://mover6_description/meshes/Joint0Coll.dae" scale="0.001 0.001 0.001"/>
+			</geometry>
+		</collision>
+		<xacro:default_inertial z_value="0" mass="1.5"/>
+	</link>
+	<link name="link1">
+		<visual>
+			<origin rpy="0 0 0" xyz="0 0 0"/>
+			<geometry>
+				<mesh filename="package://mover6_description/meshes/Joint1.dae"  scale="0.001 0.001 0.001"/>
+			</geometry>
+		</visual>
+		<collision>
+			<origin xyz="0 0 0" rpy="0 0 0" />
+			<geometry>
+				<mesh filename="package://mover6_description/meshes/Joint1Coll.dae" scale="0.001 0.001 0.001"/>
+			</geometry>
+		</collision>
+		<xacro:default_inertial z_value="0" mass="0.5"/>
+	</link>
+	<link name="link2">
+		<visual>
+			<origin rpy="0 0 0" xyz="0 0 0"/>
+			<geometry>
+				<mesh filename="package://mover6_description/meshes/Joint2.dae"  scale="0.001 0.001 0.001"/>
+			</geometry>
+		</visual>
+		<collision>
+			<origin xyz="0 0 0" rpy="0 0 0" />
+			<geometry>
+				<mesh filename="package://mover6_description/meshes/Joint2Coll.dae" scale="0.001 0.001 0.001"/>
+			</geometry>
+		</collision>
+		<xacro:default_inertial z_value="0" mass="0.5"/>
+	</link>
+	<link name="link3">
+		<visual>
+			<origin rpy="0 0 0" xyz="0 0 0"/>
+			<geometry>
+				<mesh filename="package://mover6_description/meshes/Joint3.dae"  scale="0.001 0.001 0.001"/>
+			</geometry>
+		</visual>
+		<collision>
+			<origin xyz="0 0 0" rpy="0 0 0" />
+			<geometry>
+				<mesh filename="package://mover6_description/meshes/Joint3Coll.dae" scale="0.001 0.001 0.001"/>
+			</geometry>
+		</collision>
+		<xacro:default_inertial z_value="0" mass="0.5"/>
+	</link>
+	<link name="link4">
+		<visual>
+			<origin rpy="0 0 0" xyz="0 0 0"/>
+			<geometry>
+				<mesh filename="package://mover6_description/meshes/Joint4.dae"  scale="0.001 0.001 0.001"/>
+			</geometry>
+		</visual>
+		<collision>
+			<origin xyz="0 0 0" rpy="0 0 0" />
+			<geometry>
+				<mesh filename="package://mover6_description/meshes/Joint4Coll.dae" scale="0.001 0.001 0.001"/>
+			</geometry>
+		</collision>
+		<xacro:default_inertial z_value="0" mass="0.2"/>
+	</link>
+	<link name="link5">
+		<visual>
+			<origin rpy="0 0 0" xyz="0 0 0"/>
+			<geometry>
+				<mesh filename="package://mover6_description/meshes/Joint5.dae"  scale="0.001 0.001 0.001"/>
+			</geometry>
+		</visual>
+		<collision>
+			<origin xyz="0 0 0" rpy="0 0 0" />
+			<geometry>
+				<mesh filename="package://mover6_description/meshes/Joint5Coll.dae" scale="0.001 0.001 0.001"/>
+			</geometry>
+		</collision>
+		<xacro:default_inertial z_value="0" mass="0.2"/>
+	</link>
+	<link name="link6">
+		<visual>
+			<origin rpy="0 0 0" xyz="0 0 0"/>
+			<geometry>
+				<mesh filename="package://mover6_description/meshes/Joint6.dae"  scale="0.001 0.001 0.001"/>
+			</geometry>
+		</visual>
+		<collision>
+			<origin xyz="0 0 0" rpy="0 0 0" />
+			<geometry>
+				<mesh filename="package://mover6_description/meshes/Joint6Coll.dae" scale="0.001 0.001 0.001"/>
+			</geometry>
+		</collision>
+		<xacro:default_inertial z_value="0" mass="0.1"/>
+	</link>
+	<joint name="joint1" type="revolute">
+		<axis xyz="0 0 -1"/>
+		<parent link="base_link"/>
+		<child link="link1"/>
+		<origin rpy="0 0 0" xyz="0 0 0.130"/>
+		<limit lower="-2.27" upper="2.27" effort="100" velocity="30"/>
+		<joint_properties damping="1.0" friction="10.0"/>
+	</joint>
+	<joint name="joint2" type="revolute">
+		<axis xyz="0 1 0"/>
+		<parent link="link1"/>
+		<child link="link2"/>
+		<origin rpy="0 0 0" xyz="0 0 0.0625"/>
+		<limit lower="-0.87" upper="1.05" effort="100" velocity="30"/>
+		<joint_properties damping="1.0" friction="10.0"/>
+	</joint>
+	<joint name="joint3" type="revolute">
+		<axis xyz="0 1 0"/>
+		<parent link="link2"/>
+		<child link="link3"/>
+		<origin rpy="0 1.57079632679 0" xyz="0 0 0.190"/>
+		<limit lower="-1.92" upper="1.31" effort="100" velocity="30"/>
+		<joint_properties damping="1.0" friction="10.0"/>
+	</joint>
+	<joint name="joint4" type="revolute">
+		<axis xyz="0 0 1"/>
+		<parent link="link3"/>
+		<child link="link4"/>
+		<origin rpy="0 0 0" xyz="-0.06 0 0"/>
+		<limit lower="-2.44" upper="2.44" effort="100" velocity="30"/>
+		<joint_properties damping="1.0" friction="10.0"/>
+	</joint>
+	<joint name="joint5" type="revolute">
+		<axis xyz="0 1 0"/>
+		<parent link="link4"/>
+		<child link="link5"/>
+		<origin rpy="0 0 0" xyz="0 0 0.290"/>
+		<limit lower="-1.22" upper="1.05" effort="100" velocity="40"/>
+		<joint_properties damping="1.0" friction="1.0"/>
+	</joint>
+	<joint name="joint6" type="revolute">
+		<axis xyz="0 0 1"/>
+		<parent link="link5"/>
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
Commit message: Update urdf

File: src/mover6_description/urdf/CPRMover6.urdf.xacro (robot description, xacro)
@@ -15,7 +15,7 @@
 			<origin xyz="0 0 ${z_value}" rpy="0 0 0"/>
 			<mass value="${mass}" />
-			<inertia ixx="1.0" ixy="0.0" ixz="0.0"
-               iyy="1.0" iyz="0.0"
-               izz="1.0" />
+			<inertia ixx="0.1" ixy="0.0" ixz="0.0"
+               iyy="0.1" iyz="0.0"
+               izz="0.1" />
 		</inertial>
 	</xacro:macro>

Commit message: Multi-Robot Support (#4)
* Started two robot support

* updated launch + urdf

* Multirobot support

* tweak robot placement

* Update urdf

* Update block spawner

File: src/mover6_description/urdf/CPRMover6.urdf.xacro (robot description, xacro)
@@ -15,7 +15,7 @@
 			<origin xyz="0 0 ${z_value}" rpy="0 0 0"/>
 			<mass value="${mass}" />
-			<inertia ixx="1.0" ixy="0.0" ixz="0.0"
-               iyy="1.0" iyz="0.0"
-               izz="1.0" />
+			<inertia ixx="0.1" ixy="0.0" ixz="0.0"
+               iyy="0.1" iyz="0.0"
+               izz="0.1" />
 		</inertial>
 	</xacro:macro>
@@ -235,5 +235,4 @@
     <gazebo>
     <plugin name="gazebo_ros_control" filename="libgazebo_ros_control.so">
-        <robotNamespace>/mover6</robotNamespace>
     </plugin>
     </gazebo>
