Commit message: A gripper in the simulation

File: src/mover6_description/urdf/CPRMover6.urdf.xacro (robot description, xacro)
@@ -233,4 +233,478 @@
 		</actuator>
 	</transmission>
+  <link
+    name="left_outer_knuckle">
+    <inertial>
+      <origin
+        xyz="0.0178331863169983 3.68915177224286E-11 0.0021442477325704"
+        rpy="0 0 0" />
+      <mass
+        value="0.00684838849434396" />
+      <inertia
+        ixx="2.66832029033166E-07"
+        ixy="1.66142314639824E-15"
+        ixz="1.45945633322873E-07"
+        iyy="1.3889233257419E-06"
+        iyz="2.82951161241588E-15"
+        izz="1.26603336914415E-06" />
+    </inertial>
+    <visual>
+      <origin
+        xyz="0 0 0"
+        rpy="0 0 0" />
+      <geometry>
+        <mesh
+          filename="package://robotiq_arg85_description/meshes/outer_knuckle_fine.STL" />
+      </geometry>
+      <material
+        name="">
+        <color
+          rgba="0.1 0.1 0.1 1" />
+      </material>
+    </visual>
+    <collision>
+      <origin
+        xyz="0 0 0"
+        rpy="0 0 0" />
+      <geometry>
+        <mesh
+          filename="package://robotiq_arg85_description/meshes/outer_knuckle_coarse.STL" />
+      </geometry>
+    </collision>
+  </link>
+  <joint
+    name="finger_joint"
+    type="revolute">
+    <origin
+      xyz="0.0306011444260539 0 0.0627920162695395"
+      rpy="0 0 0" />
+    <parent
+      link="link6" />
+    <child
+      link="left_outer_knuckle" />
+    <axis
+      xyz="0 -1 0" />
+    <limit
+	  lower="0"
+      upper="0.725"
+      velocity="2.0"
+      effort="1000" />
+  </joint>
+  <link
+    name="left_outer_finger">
+    <inertial>
+      <origin
+        xyz="0.00131451599174296 2.88942057994543E-15 0.0215404163180413"
+        rpy="0 0 0" />
+      <mass
+        value="0.0273093985570947" />
+      <inertia
+        ixx="8.51629628283022E-06"
+        ixy="2.58174336207405E-19"
+        ixz="3.83829504344079E-07"
+        iyy="6.9133328065108E-06"
+        iyz="-7.58589926143789E-19"
+        izz="2.25006832221981E-06" />
+    </inertial>
+    <visual>
+      <origin
+        xyz="0 0 0"
+        rpy="0 0 0" />
+      <geometry>
+        <mesh
+          filename="package://robotiq_arg85_description/meshes/outer_finger_fine.STL" />
+      </geometry>
+      <material
+        name="">
+        <color
+          rgba="0.1 0.1 0.1 1" />
+      </material>
+    </visual>
+    <collision>
+      <origin
+        xyz="0 0 0"
+        rpy="0 0 0" />
+      <geometry>
+        <mesh
+          filename="package://robotiq_arg85_description/meshes/outer_finger_coarse.STL" />
+      </geometry>
+    </collision>
+  </link>
+  <joint
+    name="left_outer_finger_joint"
+    type="fixed">
+    <origin
+      xyz="0.0316910442266543 0 -0.00193396375724605"
+      rpy="0 0 0" />
+    <parent
+      link="left_outer_knuckle" />
+    <child
+      link="left_outer_finger" />
+    <axis
+      xyz="0 -1 0" />
+  </joint>
+  <link
+    name="left_inner_knuckle">
+    <inertial>
+      <origin
+        xyz="0.017097546626628 -3.93808524389535E-10 0.0224918438201868"
+        rpy="0 0 0" />
+      <mass
+        value="0.0110930853895903" />
+      <inertia
+        ixx="4.23392770691541E-06"
+        ixy="5.748978936968E-15"
+        ixz="1.78855677119788E-06"
+        iyy="3.96548790524392E-06"
+        iyz="1.05464666369669E-14"
+        izz="3.24068002883007E-06" />
+    </inertial>
+    <visual>
+      <origin
+        xyz="0 0 0"
+        rpy="0 0 0" />
+      <geometry>
+        <mesh
+          filename="package://robotiq_arg85_description/meshes/inner_knuckle_fine.STL" />
+      </geometry>
+      <material
+        name="">
+        <color
+          rgba="0.1 0.1 0.1 1" />
+      </material>
+    </visual>
+    <collision>
+      <origin
+        xyz="0 0 0"
+        rpy="0 0 0" />
+      <geometry>
+        <mesh
+          filename="package://robotiq_arg85_description/meshes/inner_knuckle_coarse.STL" />
+      </geometry>
+    </collision>
+  </link>
+  <joint
+    name="left_inner_knuckle_joint"
+    type="revolute">
+    <origin
+      xyz="0.0127000000001501 0 0.0693074999999639"
+      rpy="0 0 0" />
+    <parent
+      link="link6" />
+    <child
+      link="left_inner_knuckle" />
+    <axis
+      xyz="0 -1 0" />
+    <limit
+      lower="0"
+      upper="0.8757"
+      velocity="2.0"
+      effort="1000" />
+    <mimic
+      joint="finger_joint"
+      multiplier="1"
+      offset="0" />
+  </joint>
+  <link
+    name="left_inner_finger">
+    <inertial>
+      <origin
+        xyz="0.0060275613594574 -6.29183141465421E-15 0.00669925693133241"
+        rpy="0 0 0" />
+      <mass
+        value="0.00724255346165745" />
+      <inertia
+        ixx="1.47824274053603E-06"
+        ixy="-3.94884463570303E-19"
+        ixz="-3.45268847648622E-07"
+        iyy="1.70064480838395E-06"
+        iyz="3.5059838910097E-19"
+        izz="4.77151336838364E-07" />
+    </inertial>
+    <visual>
+      <origin
+        xyz="0 0 0"
+        rpy="0 0 0" />
+      <geometry>
+        <mesh
+          filename="package://robotiq_arg85_description/meshes/inner_finger_fine.STL" />
+      </geometry>
+      <material
+        name="">
+        <color
+          rgba="0.1 0.1 0.1 1" />
+      </material>
+    </visual>
+    <collision>
+      <origin
+        xyz="0 0 0"
+        rpy="0 0 0" />
+      <geometry>
+        <mesh
+          filename="package://robotiq_arg85_description/meshes/inner_finger_coarse.STL" />
+      </geometry>
+    </collision>
+  </link>
+  <joint
+    name="left_inner_finger_joint"
+    type="revolute">
+    <origin
+      xyz="0.034585310861294 0 0.0454970193817975"
+      rpy="0 0 0" />
+    <parent
+      link="left_inner_knuckle" />
+    <child
+      link="left_inner_finger" />
+    <axis
+      xyz="0 -1 0" />
+    <limit
+      lower="0"
+      upper="0.8757"
+      velocity="2.0"
+      effort="1000" />
+    <mimic
+      joint="finger_joint"
+      multiplier="-1"
+      offset="0" />
+  </joint>
+  <link
+    name="right_inner_knuckle">
+    <inertial>
+      <origin
+        xyz="0.0168606186773776 3.93808471820465E-10 0.0226699950793434"
+        rpy="0 0 0" />
+      <mass
+        value="0.0110930853895903" />
+      <inertia
+        ixx="4.27134775939882E-06"
+        ixy="-8.53568456728898E-15"
+        ixz="1.77774229944246E-06"
+        iyy="3.96548790524392E-06"
+        iyz="-8.45108024914164E-15"
+        izz="3.20325997634666E-06" />
+    </inertial>
+    <visual>
+      <origin
+        xyz="0 0 0"
+        rpy="0 0 0" />
+      <geometry>
+        <mesh
+          filename="package://robotiq_arg85_description/meshes/inner_knuckle_fine.STL" />
+      </geometry>
+      <material
+        name="">
+        <color
+          rgba="0.1 0.1 0.1 1" />
+      </material>
+    </visual>
+    <collision>
+      <origin
+        xyz="0 0 0"
+        rpy="0 0 0" />
+      <geometry>
+        <mesh
+          filename="package://robotiq_arg85_description/meshes/inner_knuckle_coarse.STL" />
+      </geometry>
+    </collision>
+  </link>
+  <joint
+    name="right_inner_knuckle_joint"
+    type="revolute">
+    <origin
+      xyz="-0.0126999999998499 0 0.0693075000000361"
+      rpy="0 0 3.14159265358979" />
+    <parent
+      link="link6" />
+    <child
+      link="right_inner_knuckle" />
+    <axis
+      xyz="0 1 0" />
+    <limit
+      lower="0"
+      upper="0.8757"
+      velocity="2.0"
+      effort="1000" />
+    <mimic
+      joint="finger_joint"
+      multiplier="-1"
+      offset="0" />
+  </joint>
+  <link
+    name="right_inner_finger">
+    <inertial>
+      <origin
+        xyz="0.00602756228812038 -6.47284509480176E-15 0.00669925609578108"
+        rpy="0 0 0" />
+      <mass
+        value="0.00724255346165744" />
+      <inertia
+        ixx="1.47824283625957E-06"
+        ixy="-3.95952064019123E-19"
+        ixz="-3.45268708875543E-07"
+        iyy="1.70064480838394E-06"
+        iyz="3.55286507960029E-19"
+        izz="4.77151241114822E-07" />
+    </inertial>
+    <visual>
+      <origin
+        xyz="0 0 0"
+        rpy="0 0 0" />
+      <geometry>
+        <mesh
+          filename="package://robotiq_arg85_description/meshes/inner_finger_fine.STL" />
+      </geometry>
+      <material
+        name="">
+        <color
+          rgba="0.1 0.1 0.1 1" />
+      </material>
+    </visual>
+    <collision>
+      <origin
+        xyz="0 0 0"
+        rpy="0 0 0" />
+      <geometry>
+        <mesh
+          filename="package://robotiq_arg85_description/meshes/inner_finger_coarse.STL" />
+      </geometry>
+    </collision>
+  </link>
+  <joint
+    name="right_inner_finger_joint"
+    type="revolute">
+    <origin
+      xyz="0.0341060475457406 0 0.0458573878541688"
+      rpy="0 0 0" />
+    <parent
+      link="right_inner_knuckle" />
+    <child
+      link="right_inner_finger" />
+    <axis
+      xyz="0 1 0" />
+    <limit
+      lower="0"
+      upper="0.8757"
+      velocity="2.0"
+      effort="1000" />
+    <mimic
+      joint="finger_joint"
+      multiplier="1"
+      offset="0" />
+  </joint>
+  <link
+    name="right_outer_knuckle">
+    <inertial>
+      <origin
+        xyz="0.0178097074051638 3.60493211424024E-11 0.00233123458346721"
+        rpy="0 0 0" />
+      <mass
+        value="0.00684838849401352" />
+      <inertia
+        ixx="2.70004361573169E-07"
+        ixy="1.59579467624491E-15"
+        ixz="1.56396493788199E-07"
+        iyy="1.38892332558312E-06"
+        iyz="2.82357800318817E-15"
+        izz="1.26286103637978E-06" />
+    </inertial>
+    <visual>
+      <origin
+        xyz="0 0 0"
+        rpy="0 0 0" />
+      <geometry>
+        <mesh
+          filename="package://robotiq_arg85_description/meshes/outer_knuckle_fine.STL" />
+      </geometry>
+      <material
+        name="">
+        <color
+          rgba="0.1 0.1 0.1 1" />
+      </material>
+    </visual>
+    <collision>
+      <origin
+        xyz="0 0 0"
+        rpy="0 0 0" />
+      <geometry>
+        <mesh
+          filename="package://robotiq_arg85_description/meshes/outer_knuckle_coarse.STL" />
+      </geometry>
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
Commit message: Add gripper mount

File: src/mover6_description/urdf/CPRMover6.urdf.xacro (robot description, xacro)
@@ -233,4 +233,49 @@
 		</actuator>
 	</transmission>
+<link
+    name="robotiq_85_base_link">
+    <inertial>
+      <origin
+        xyz="0.00021987 -2.3546E-10 0.030163"
+        rpy="0 0 0" />
+      <mass
+        value="0.30915" />
+      <inertia
+        ixx="0.00028972"
+        ixy="-5.7879E-10"
+        ixz="-1.8543E-06"
+        iyy="0.00030737"
+        iyz="1.682E-12"
+        izz="0.00019914" />
+    </inertial>
+    <visual>
+      <origin
+        xyz="0 0 0"
+        rpy="0 0 0" />
+      <geometry>
+        <mesh
+          filename="package://robotiq_arg85_description/meshes/robotiq_85_base_link_fine.STL" />
+      </geometry>
+      <material
+        name="">
+        <color
+          rgba="0.1 0.1 0.1 1" />
+      </material>
+    </visual>
+    <collision>
+      <origin
+        xyz="0 0 0"
+        rpy="0 0 0" />
+      <geometry>
+        <mesh
+          filename="package://robotiq_arg85_description/meshes/robotiq_85_base_link_coarse.STL" />
+      </geometry>
+    </collision>
+  </link>
+  <joint name="gripper_mount" type="fixed">
+    <parent link="link6"/>
+    <child link="robotiq_85_base_link"/>
+    <origin xyz="0 0 0"/>
+  </joint>
   <link
     name="left_outer_knuckle">
@@ -280,5 +325,5 @@
       rpy="0 0 0" />
     <parent
-      link="link6" />
+      link="robotiq_85_base_link" />
     <child
       link="left_outer_knuckle" />
@@ -391,5 +436,5 @@
       rpy="0 0 0" />
     <parent
-      link="link6" />
+      link="robotiq_85_base_link" />
     <child
       link="left_inner_knuckle" />
@@ -515,5 +560,5 @@
       rpy="0 0 3.14159265358979" />
     <parent
-      link="link6" />
+      link="robotiq_85_base_link" />
     <child
       link="right_inner_knuckle" />
@@ -639,5 +684,5 @@
       rpy="0 0 3.14159265358979" />
     <parent
-      link="link6" />
+      link="robotiq_85_base_link" />
     <child
       link="right_outer_knuckle" />

Commit message: Change scale + fix invkin

File: src/mover6_description/urdf/CPRMover6.urdf.xacro (robot description, xacro)
@@ -255,19 +255,19 @@
       <geometry>
         <mesh
-          filename="package://robotiq_arg85_description/meshes/robotiq_85_base_link_fine.STL" />
-      </geometry>
-      <material
-        name="">
-        <color
-          rgba="0.1 0.1 0.1 1" />
-      </material>
-    </visual>
-    <collision>
-      <origin
-        xyz="0 0 0"
-        rpy="0 0 0" />
-      <geometry>
-        <mesh
-          filename="package://robotiq_arg85_description/meshes/robotiq_85_base_link_coarse.STL" />
+          filename="package://robotiq_arg85_description/meshes/robotiq_85_base_link_fine.STL" scale="0.5 0.5 0.5"/>
+      </geometry>
+      <material
+        name="">
+        <color
+          rgba="0.1 0.1 0.1 1" />
+      </material>
+    </visual>
+    <collision>
+      <origin
+        xyz="0 0 0"
+        rpy="0 0 0" />
+      <geometry>
+        <mesh
+          filename="package://robotiq_arg85_description/meshes/robotiq_85_base_link_coarse.STL" scale="0.5 0.5 0.5"/>
       </geometry>
     </collision>
@@ -300,19 +300,19 @@
       <geometry>
         <mesh
-          filename="package://robotiq_arg85_description/meshes/outer_knuckle_fine.STL" />
-      </geometry>
-      <material
-        name="">
-        <color
-          rgba="0.1 0.1 0.1 1" />
-      </material>
-    </visual>
-    <collision>
-      <origin
-        xyz="0 0 0"
-        rpy="0 0 0" />
-      <geometry>
-        <mesh
-          filename="package://robotiq_arg85_description/meshes/outer_knuckle_coarse.STL" />
+          filename="package://robotiq_arg85_description/meshes/outer_knuckle_fine.STL" scale="0.5 0.5 0.5"/>
+      </geometry>
+      <material
+        name="">
+        <color
+          rgba="0.1 0.1 0.1 1" />
+      </material>
+    </visual>
+    <collision>
+      <origin
+        xyz="0 0 0"
+        rpy="0 0 0" />
+      <geometry>
+        <mesh
+          filename="package://robotiq_arg85_description/meshes/outer_knuckle_coarse.STL" scale="0.5 0.5 0.5"/>
       </geometry>
     </collision>
@@ -358,19 +358,19 @@
       <geometry>
         <mesh
-          filename="package://robotiq_arg85_description/meshes/outer_finger_fine.STL" />
-      </geometry>
-      <material
-        name="">
-        <color
-          rgba="0.1 0.1 0.1 1" />
-      </material>
-    </visual>
-    <collision>
-      <origin
-        xyz="0 0 0"
-        rpy="0 0 0" />
-      <geometry>
-        <mesh
-          filename="package://robotiq_arg85_description/meshes/outer_finger_coarse.STL" />
+          filename="package://robotiq_arg85_description/meshes/outer_finger_fine.STL" scale="0.5 0.5 0.5"/>
+      </geometry>
+      <material
+        name="">
+        <color
+          rgba="0.1 0.1 0.1 1" />
+      </material>
+    </visual>
+    <collision>
+      <origin
+        xyz="0 0 0"
+        rpy="0 0 0" />
+      <geometry>
+        <mesh
+          filename="package://robotiq_arg85_description/meshes/outer_finger_coarse.STL" scale="0.5 0.5 0.5"/>
       </geometry>
     </collision>
@@ -378,5 +378,5 @@
   <joint
     name="left_outer_finger_joint"
-    type="fixed">
+    type="revolute">
     <origin
       xyz="0.0316910442266543 0 -0.00193396375724605"
@@ -388,4 +388,9 @@
     <axis
       xyz="0 -1 0" />
+    <limit
+	  lower="0"
+      upper="0"
+      velocity="0"
+      effort="0" />
   </joint>
   <link
@@ -411,19 +416,19 @@
       <geometry>
         <mesh
-          filename="package://robotiq_arg85_description/meshes/inner_knuckle_fine.STL" />
-      </geometry>
-      <material
-        name="">
-        <color
-          rgba="0.1 0.1 0.1 1" />
-      </material>
-    </visual>
-    <collision>
-      <origin
-        xyz="0 0 0"
-        rpy="0 0 0" />
-      <geometry>
-        <mesh
-          filename="package://robotiq_arg85_description/meshes/inner_knuckle_coarse.STL" />
+          filename="package://robotiq_arg85_description/meshes/inner_knuckle_fine.STL" scale="0.5 0.5 0.5"/>
+      </geometry>
+      <material
+        name="">
+        <color
+          rgba="0.1 0.1 0.1 1" />
+      </material>
+    </visual>
+    <collision>
+      <origin
+        xyz="0 0 0"
+        rpy="0 0 0" />
+      <geometry>
+        <mesh
+          filename="package://robotiq_arg85_description/meshes/inner_knuckle_coarse.STL" scale="0.5 0.5 0.5"/>
       </geometry>
     </collision>
@@ -473,19 +478,19 @@
       <geometry>
         <mesh
-          filename="package://robotiq_arg85_description/meshes/inner_finger_fine.STL" />
-      </geometry>
-      <material
-        name="">
-        <color
-          rgba="0.1 0.1 0.1 1" />
-      </material>
-    </visual>
-    <collision>
-      <origin
-        xyz="0 0 0"
-        rpy="0 0 0" />
-      <geometry>
-        <mesh
-          filename="package://robotiq_arg85_description/meshes/inner_finger_coarse.STL" />
+          filename="package://robotiq_arg85_description/meshes/inner_finger_fine.STL" scale="0.5 0.5 0.5"/>
+      </geometry>
+      <material
+        name="">
+        <color
+          rgba="0.1 0.1 0.1 1" />
+      </material>
+    </visual>
+    <collision>
+      <origin
+        xyz="0 0 0"
+        rpy="0 0 0" />
+      <geometry>
+        <mesh
+          filename="package://robotiq_arg85_description/meshes/inner_finger_coarse.STL" scale="0.5 0.5 0.5"/>
       </geometry>
     </collision>
@@ -535,19 +540,19 @@
       <geometry>
         <mesh
-          filename="package://robotiq_arg85_description/meshes/inner_knuckle_fine.STL" />
-      </geometry>
-      <material
-        name="">
-        <color
-          rgba="0.1 0.1 0.1 1" />
-      </material>
-    </visual>
-    <collision>
-      <origin
-        xyz="0 0 0"
-        rpy="0 0 0" />
-      <geometry>
-        <mesh
-          filename="package://robotiq_arg85_description/meshes/inner_knuckle_coarse.STL" />
+          filename="package://robotiq_arg85_description/meshes/inner_knuckle_fine.STL" scale="0.5 0.5 0.5"/>
+      </geometry>
+      <material
+        name="">
+        <color
+          rgba="0.1 0.1 0.1 1" />
+      </material>
+    </visual>
+    <collision>
+      <origin
+        xyz="0 0 0"
+        rpy="0 0 0" />
+      <geometry>
+        <mesh
+          filename="package://robotiq_arg85_description/meshes/inner_knuckle_coarse.STL" scale="0.5 0.5 0.5"/>
       </geometry>
     </collision>
@@ -597,19 +602,19 @@
       <geometry>
         <mesh
-          filename="package://robotiq_arg85_description/meshes/inner_finger_fine.STL" />
-      </geometry>
-      <material
-        name="">
-        <color
-          rgba="0.1 0.1 0.1 1" />
-      </material>
-    </visual>
-    <collision>
-      <origin
-        xyz="0 0 0"
-        rpy="0 0 0" />
-      <geometry>
-        <mesh
-          filename="package://robotiq_arg85_description/meshes/inner_finger_coarse.STL" />
+          filename="package://robotiq_arg85_description/meshes/inner_finger_fine.STL" scale="0.5 0.5 0.5"/>
+      </geometry>
+      <material
+        name="">
+        <color
+          rgba="0.1 0.1 0.1 1" />
+      </material>
+    </visual>
+    <collision>
+      <origin
+        xyz="0 0 0"
+        rpy="0 0 0" />
+      <geometry>
+        <mesh
+          filename="package://robotiq_arg85_description/meshes/inner_finger_coarse.STL" scale="0.5 0.5 0.5"/>
       </geometry>
     </collision>
@@ -659,19 +664,19 @@
       <geometry>
         <mesh
-          filename="package://robotiq_arg85_description/meshes/outer_knuckle_fine.STL" />
-      </geometry>
-      <material
-        name="">
-        <color
-          rgba="0.1 0.1 0.1 1" />
-      </material>
-    </visual>
-    <collision>
-      <origin
-        xyz="0 0 0"
-        rpy="0 0 0" />
-      <geometry>
-        <mesh
-          filename="package://robotiq_arg85_description/meshes/outer_knuckle_coarse.STL" />
+          filename="package://robotiq_arg85_description/meshes/outer_knuckle_fine.STL" scale="0.5 0.5 0.5"/>
+      </geometry>
+      <material
+        name="">
+        <color
+          rgba="0.1 0.1 0.1 1" />
+      </material>
+    </visual>
+    <collision>
+      <origin
+        xyz="0 0 0"
+        rpy="0 0 0" />
+      <geometry>
+        <mesh
+          filename="package://robotiq_arg85_description/meshes/outer_knuckle_coarse.STL" scale="0.5 0.5 0.5"/>
       </geometry>
     </collision>
@@ -721,19 +726,19 @@
       <geometry>
         <mesh
-          filename="package://robotiq_arg85_description/meshes/outer_finger_fine.STL" />
-      </geometry>
-      <material
-        name="">
-        <color
-          rgba="0.1 0.1 0.1 1" />
-      </material>
-    </visual>
-    <collision>
-      <origin
-        xyz="0 0 0"
-        rpy="0 0 0" />
-      <geometry>
-        <mesh
-          filename="package://robotiq_arg85_description/meshes/outer_finger_coarse.STL" />
+          filename="package://robotiq_arg85_description/meshes/outer_finger_fine.STL" scale="0.5 0.5 0.5"/>
+      </geometry>
+      <material
+        name="">
+        <color
+          rgba="0.1 0.1 0.1 1" />
+      </material>
+    </visual>
+    <collision>
+      <origin
+        xyz="0 0 0"
+        rpy="0 0 0" />
+      <geometry>
+        <mesh
+          filename="package://robotiq_arg85_description/meshes/outer_finger_coarse.STL" scale="0.5 0.5 0.5"/>
       </geometry>
     </collision>
@@ -741,5 +746,5 @@
   <joint
     name="right_outer_finger_joint"
-    type="fixed">
+    type="revolute">
     <origin
       xyz="0.0317095909367246 0 -0.0016013564954687"
@@ -751,4 +756,9 @@
     <axis
       xyz="0 1 0" />
+    <limit
+	  lower="0"
+      upper="0"
+      velocity="0"
+      effort="0" />
   </joint>
     <gazebo>
