Commit message: Gripper control beginings

File: src/mover6_description/urdf/CPRMover6.urdf.xacro (robot description, xacro)
@@ -233,4 +233,14 @@
 		</actuator>
 	</transmission>
+	<transmission name="tran7">
+		<type>transmission_interface/SimpleTransmission</type>
+		<joint name="finger_joint">
+			<hardwareInterface>hardware_interface/EffortJointInterface</hardwareInterface>
+		</joint>
+		<actuator name="motor7">
+		    <hardwareInterface>hardware_interface/EffortJointInterface</hardwareInterface>
+			<mechanicalReduction>1</mechanicalReduction>
+		</actuator>
+	</transmission>
 <link
     name="robotiq_85_base_link">
@@ -241,11 +251,11 @@
       <mass
         value="0.30915" />
-      <inertia
-        ixx="0.00028972"
-        ixy="-5.7879E-10"
-        ixz="-1.8543E-06"
-        iyy="0.00030737"
-        iyz="1.682E-12"
-        izz="0.00019914" />
+    <inertia
+        ixx="0.0001"
+        ixy="0.000"
+        ixz="0.000"
+        iyy="0.0001"
+        iyz="0.000"
+        izz="0.0001"/>
     </inertial>
     <visual>
@@ -286,11 +296,11 @@
       <mass
         value="0.00684838849434396" />
-      <inertia
-        ixx="2.66832029033166E-07"
-        ixy="1.66142314639824E-15"
-        ixz="1.45945633322873E-07"
-        iyy="1.3889233257419E-06"
-        iyz="2.82951161241588E-15"
-        izz="1.26603336914415E-06" />
+    <inertia
+        ixx="0.0001"
+        ixy="0.000"
+        ixz="0.000"
+        iyy="0.0001"
+        iyz="0.000"
+        izz="0.0001"/>
     </inertial>
     <visual>
@@ -344,11 +354,11 @@
       <mass
         value="0.0273093985570947" />
-      <inertia
-        ixx="8.51629628283022E-06"
-        ixy="2.58174336207405E-19"
-        ixz="3.83829504344079E-07"
-        iyy="6.9133328065108E-06"
-        iyz="-7.58589926143789E-19"
-        izz="2.25006832221981E-06" />
+    <inertia
+        ixx="0.0001"
+        ixy="0.000"
+        ixz="0.000"
+        iyy="0.0001"
+        iyz="0.000"
+        izz="0.0001"/>
     </inertial>
     <visual>
@@ -402,11 +412,11 @@
       <mass
         value="0.0110930853895903" />
-      <inertia
-        ixx="4.23392770691541E-06"
-        ixy="5.748978936968E-15"
-        ixz="1.78855677119788E-06"
-        iyy="3.96548790524392E-06"
-        iyz="1.05464666369669E-14"
-        izz="3.24068002883007E-06" />
+    <inertia
+        ixx="0.0001"
+        ixy="0.000"
+        ixz="0.000"
+        iyy="0.0001"
+        iyz="0.000"
+        izz="0.0001"/>
     </inertial>
     <visual>
@@ -464,11 +474,11 @@
       <mass
         value="0.00724255346165745" />
-      <inertia
-        ixx="1.47824274053603E-06"
-        ixy="-3.94884463570303E-19"
-        ixz="-3.45268847648622E-07"
-        iyy="1.70064480838395E-06"
-        iyz="3.5059838910097E-19"
-        izz="4.77151336838364E-07" />
+    <inertia
+        ixx="0.0001"
+        ixy="0.000"
+        ixz="0.000"
+        iyy="0.0001"
+        iyz="0.000"
+        izz="0.0001"/>
     </inertial>
     <visual>
@@ -526,11 +536,11 @@
       <mass
         value="0.0110930853895903" />
-      <inertia
-        ixx="4.27134775939882E-06"
-        ixy="-8.53568456728898E-15"
-        ixz="1.77774229944246E-06"
-        iyy="3.96548790524392E-06"
-        iyz="-8.45108024914164E-15"
-        izz="3.20325997634666E-06" />
+    <inertia
+        ixx="0.0001"
+        ixy="0.000"
+        ixz="0.000"
+        iyy="0.0001"
+        iyz="0.000"
+        izz="0.0001"/>
     </inertial>
     <visual>
@@ -588,11 +598,11 @@
       <mass
         value="0.00724255346165744" />
-      <inertia
-        ixx="1.47824283625957E-06"
-        ixy="-3.95952064019123E-19"
-        ixz="-3.45268708875543E-07"
-        iyy="1.70064480838394E-06"
-        iyz="3.55286507960029E-19"
-        izz="4.77151241114822E-07" />
+    <inertia
+        ixx="0.0001"
+        ixy="0.000"
+        ixz="0.000"
+        iyy="0.0001"
+        iyz="0.000"
+        izz="0.0001"/>
     </inertial>
     <visual>
@@ -650,11 +660,11 @@
       <mass
         value="0.00684838849401352" />
-      <inertia
-        ixx="2.70004361573169E-07"
-        ixy="1.59579467624491E-15"
-        ixz="1.56396493788199E-07"
-        iyy="1.38892332558312E-06"
-        iyz="2.82357800318817E-15"
-        izz="1.26286103637978E-06" />
+    <inertia
+        ixx="0.0001"
+        ixy="0.000"
+        ixz="0.000"
+        iyy="0.0001"
+        iyz="0.000"
+        izz="0.0001"/>
     </inertial>
     <visual>
@@ -712,11 +722,11 @@
       <mass
         value="0.0273093985570947" />
-      <inertia
-        ixx="8.52366028592721E-06"
-        ixy="3.41683380899422E-19"
-        ixz="3.18003675694284E-07"
-        iyy="6.91333280651081E-06"
-        iyz="7.37726682706417E-19"
-        izz="2.24270431912283E-06" />
+    <inertia
+        ixx="0.0001"
+        ixy="0.000"
+        ixz="0.000"
+        iyy="0.0001"
+        iyz="0.000"
+        izz="0.0001"/>
     </inertial>
     <visual>
@@ -762,4 +772,31 @@
       effort="0" />
   </joint>
+    <gazebo reference="gripper_mount">
+        <selfCollide>False</selfCollide>
+    </gazebo>
+    <gazebo reference="finger_joint">
+        <selfCollide>False</selfCollide>
+    </gazebo>
+    <gazebo reference="left_outer_finger_joint">
+        <selfCollide>False</selfCollide>
+    </gazebo>
+    <gazebo reference="left_inner_knuckle_joint">
+        <selfCollide>False</selfCollide>
+    </gazebo>
+    <gazebo reference="left_inner_finger_joint">
+        <selfCollide>False</selfCollide>
+    </gazebo>
+    <gazebo reference="right_inner_knuckle_joint">
+        <selfCollide>False</selfCollide>
+    </gazebo>
+    <gazebo reference="right_inner_finger_joint">
+        <selfCollide>False</selfCollide>
+    </gazebo>
+    <gazebo reference="right_outer_knuckle_joint">
+        <selfCollide>False</selfCollide>
+    </gazebo>
+    <gazebo reference="right_outer_finger_joint">
+        <selfCollide>False</selfCollide>
+    </gazebo>
     <gazebo>
     <plugin name="gazebo_ros_control" filename="libgazebo_ros_control.so">

Commit message: Playing with tf

File: src/mover6_description/urdf/CPRMover6.urdf.xacro (robot description, xacro)
@@ -5,9 +5,4 @@
 	<!-- Version 1.1 from Oct. 04th, 2016. -->
 	<!-- Used for fixing robot to Gazebo 'base_link' -->
-	<link name="world"/>
-	<joint name="fixed" type="fixed">
-		<parent link="world"/>
-		<child link="base_link"/>
-	</joint>
 	<!-- Default Inertial -->
 	<xacro:macro name="default_inertial" params="z_value mass">

Commit message: Slow down sim robots

File: src/mover6_description/urdf/CPRMover6.urdf.xacro (robot description, xacro)
@@ -15,7 +15,7 @@
 			<origin xyz="0 0 ${z_value}" rpy="0 0 0"/>
 			<mass value="${mass}" />
-			<inertia ixx="0.1" ixy="0.0" ixz="0.0"
-               iyy="0.1" iyz="0.0"
-               izz="0.1" />
+			<inertia ixx="0.01" ixy="0.0" ixz="0.0"
+               iyy="0.01" iyz="0.0"
+               izz="0.01" />
 		</inertial>
 	</xacro:macro>

Commit message: gripper in simulation, angles need figuring out

File: src/mover6_description/urdf/CPRMover6.urdf.xacro (robot description, xacro)
@@ -125,4 +125,49 @@
 		<xacro:default_inertial z_value="0" mass="0.1"/>
 	</link>
+	<link name="link7">
+		<visual>
+			<origin rpy="0 0 0" xyz="0 0 0"/>
+			<geometry>
+				<mesh filename="package://mover6_description/meshes/joint7.STL"  scale="1 1 1"/>
+			</geometry>
+		</visual>
+		<collision>
+			<origin xyz="0 0 0" rpy="0 0 0" />
+			<geometry>
+				<mesh filename="package://mover6_description/meshes/joint7.STL" scale="1 1 1"/>
+			</geometry>
+		</collision>
+		<xacro:default_inertial z_value="0" mass="0.1"/>
+	</link>
+	<link name="gripper_a">
+		<visual>
+			<origin rpy="0 0 0" xyz="0 0 0"/>
+			<geometry>
+				<mesh filename="package://mover6_description/meshes/gripper_a.STL"  scale="1 1 1"/>
+			</geometry>
+		</visual>
+		<collision>
+			<origin xyz="0 0 0" rpy="0 0 0" />
+			<geometry>
+				<mesh filename="package://mover6_description/meshes/gripper_a.STL" scale="1 1 1"/>
+			</geometry>
+		</collision>
+		<xacro:default_inertial z_value="0" mass="0.1"/>
+	</link>
+	<link name="gripper_b">
+		<visual>
+			<origin rpy="0 0 0" xyz="0 0 0"/>
+			<geometry>
+				<mesh filename="package://mover6_description/meshes/gripper_b.STL"  scale="1 1 1"/>
+			</geometry>
+		</visual>
+		<collision>
+			<origin xyz="0 0 0" rpy="0 0 0" />
+			<geometry>
+				<mesh filename="package://mover6_description/meshes/gripper_b.STL" scale="1 1 1"/>
+			</geometry>
+		</collision>
+		<xacro:default_inertial z_value="0" mass="0.1"/>
+	</link>
 	<joint name="joint1" type="revolute">
 		<axis xyz="0 0 -1"/>
@@ -173,4 +218,28 @@
 		<joint_properties damping="1.0" friction="1.0"/>
 	</joint>
+	<joint name="joint7" type="revolute">
+		<axis xyz="0 0 1"/>
+		<parent link="link6"/>
+		<child link="link7"/>
+		<origin rpy="0 0 0" xyz="0 0 0"/>
+		<limit lower="-2.09" upper="2.09" effort="100" velocity="100"/>
+		<joint_properties damping="1.0" friction="1.0"/>
+	</joint>
+	<joint name="joint_gripper_a" type="revolute">
+		<axis xyz="0 0 1"/>
+		<parent link="link7"/>
+		<child link="gripper_a"/>
+		<origin rpy="0 1 0" xyz="0 0 0"/>
+		<limit lower="-2.09" upper="2.09" effort="100" velocity="100"/>
+		<joint_properties damping="1.0" friction="1.0"/>
+	</joint>
+	<joint name="joint_gripper_b" type="revolute">
+		<axis xyz="0 0 1"/>
+		<parent link="link7"/>
+		<child link="gripper_b"/>
+		<origin rpy="0 0 1" xyz="0 0 0"/>
+		<limit lower="-2.09" upper="2.09" effort="100" velocity="100"/>
+		<joint_properties damping="1.0" friction="1.0"/>
+	</joint>
 	<transmission name="tran1">
 		<type>transmission_interface/SimpleTransmission</type>
@@ -229,4 +298,24 @@
 		</joint>
 		<actuator name="motor6">
+		    <hardwareInterface>hardware_interface/EffortJointInterface</hardwareInterface>
+			<mechanicalReduction>1</mechanicalReduction>
+		</actuator>
+	</transmission>
+	<transmission name="tran7">
+		<type>transmission_interface/SimpleTransmission</type>
+		<joint name="joint_gripper_a">
+			<hardwareInterface>hardware_interface/EffortJointInterface</hardwareInterface>
+		</joint>
+		<actuator name="motor7">
+		    <hardwareInterface>hardware_interface/EffortJointInterface</hardwareInterface>
+			<mechanicalReduction>1</mechanicalReduction>
+		</actuator>
+	</transmission>
+	<transmission name="tran8">
+		<type>transmission_interface/SimpleTransmission</type>
+		<joint name="joint_gripper_b">
+			<hardwareInterface>hardware_interface/EffortJointInterface</hardwareInterface>
+		</joint>
+		<actuator name="gripper_b">
 		    <hardwareInterface>hardware_interface/EffortJointInterface</hardwareInterface>
 			<mechanicalReduction>1</mechanicalReduction>

Commit message: gripper in position

File: src/mover6_description/urdf/CPRMover6.urdf.xacro (robot description, xacro)
@@ -222,22 +222,22 @@
 		<parent link="link6"/>
 		<child link="link7"/>
-		<origin rpy="0 0 0" xyz="0 0 0"/>
+		<origin rpy="3.14159 0 1.5708" xyz="0 0 0"/>
 		<limit lower="-2.09" upper="2.09" effort="100" velocity="100"/>
 		<joint_properties damping="1.0" friction="1.0"/>
 	</joint>
 	<joint name="joint_gripper_a" type="revolute">
-		<axis xyz="0 0 1"/>
+		<axis xyz="0 0 0"/>
 		<parent link="link7"/>
 		<child link="gripper_a"/>
-		<origin rpy="0 1 0" xyz="0 0 0"/>
-		<limit lower="-2.09" upper="2.09" effort="100" velocity="100"/>
+		<origin rpy="1.5708 -0.33752 3.1416" xyz="-0.0055607 -0.0041434 -0.04688"/>
+		<limit lower="0" upper="0" effort="100" velocity="100"/>
 		<joint_properties damping="1.0" friction="1.0"/>
 	</joint>
 	<joint name="joint_gripper_b" type="revolute">
-		<axis xyz="0 0 1"/>
+		<axis xyz="0 0 0"/>
 		<parent link="link7"/>
 		<child link="gripper_b"/>
-		<origin rpy="0 0 1" xyz="0 0 0"/>
-		<limit lower="-2.09" upper="2.09" effort="100" velocity="100"/>
+		<origin rpy="1.5708 -0.33752 0" xyz="0.0055607 0.005 -0.04688"/>
+		<limit lower="0" upper="0" effort="100" velocity="100"/>
 		<joint_properties damping="1.0" friction="1.0"/>
 	</joint>

Commit message: finished urdf

File: src/mover6_description/urdf/CPRMover6.urdf.xacro (robot description, xacro)
@@ -218,5 +218,5 @@
 		<joint_properties damping="1.0" friction="1.0"/>
 	</joint>
-	<joint name="joint7" type="revolute">
+	<joint name="joint7" type="fixed">
 		<axis xyz="0 0 1"/>
 		<parent link="link6"/>
@@ -231,5 +231,5 @@
 		<child link="gripper_a"/>
 		<origin rpy="1.5708 -0.33752 3.1416" xyz="-0.0055607 -0.0041434 -0.04688"/>
-		<limit lower="0" upper="0" effort="100" velocity="100"/>
+		<limit lower="-1" upper="1" effort="100" velocity="100"/>
 		<joint_properties damping="1.0" friction="1.0"/>
 	</joint>
@@ -239,5 +239,5 @@
 		<child link="gripper_b"/>
 		<origin rpy="1.5708 -0.33752 0" xyz="0.0055607 0.005 -0.04688"/>
-		<limit lower="0" upper="0" effort="100" velocity="100"/>
+		<limit lower="-1" upper="1" effort="100" velocity="100"/>
 		<joint_properties damping="1.0" friction="1.0"/>
 	</joint>

Commit message: gripper control working

File: src/mover6_description/urdf/CPRMover6.urdf.xacro (robot description, xacro)
@@ -227,5 +227,5 @@
 	</joint>
 	<joint name="joint_gripper_a" type="revolute">
-		<axis xyz="0 0 0"/>
+		<axis xyz="0 0 1"/>
 		<parent link="link7"/>
 		<child link="gripper_a"/>
@@ -235,5 +235,5 @@
 	</joint>
 	<joint name="joint_gripper_b" type="revolute">
-		<axis xyz="0 0 0"/>
+		<axis xyz="0 0 1"/>
 		<parent link="link7"/>
 		<child link="gripper_b"/>

Commit message: Sim Gripper V2 (#25)
* Initial URDF Upload

* Rename package

* Rename file paths

* updated gripper model

* gripper in simulation, angles need figuring out

* stl files

* gripper in position

* finished urdf

* gripper control working

* Tidy up

* start of open/close

* one day everything will commit at once

* open and close scripts

* maybe working open and close gripper in sim

* working gripper

* Remove changes to pickup

* Updates to grippper controller

---------

Co-authored-by: DhagonHunt <andrei.codin10@gmail.com>
Co-authored-by: tomrrr <tomtommrichards@gmail.com>

File: src/mover6_description/urdf/CPRMover6.urdf.xacro (robot description, xacro)
@@ -125,4 +125,49 @@
 		<xacro:default_inertial z_value="0" mass="0.1"/>
 	</link>
+	<link name="link7">
+		<visual>
+			<origin rpy="0 0 0" xyz="0 0 0"/>
+			<geometry>
+				<mesh filename="package://mover6_description/meshes/joint7.STL"  scale="1 1 1"/>
+			</geometry>
+		</visual>
+		<collision>
+			<origin xyz="0 0 0" rpy="0 0 0" />
+			<geometry>
+				<mesh filename="package://mover6_description/meshes/joint7.STL" scale="1 1 1"/>
+			</geometry>
+		</collision>
+		<xacro:default_inertial z_value="0" mass="0.1"/>
+	</link>
+	<link name="gripper_a">
+		<visual>
+			<origin rpy="0 0 0" xyz="0 0 0"/>
+			<geometry>
+				<mesh filename="package://mover6_description/meshes/gripper_a.STL"  scale="1 1 1"/>
+			</geometry>
+		</visual>
+		<collision>
+			<origin xyz="0 0 0" rpy="0 0 0" />
+			<geometry>
+				<mesh filename="package://mover6_description/meshes/gripper_a.STL" scale="1 1 1"/>
+			</geometry>
+		</collision>
+		<xacro:default_inertial z_value="0" mass="0.1"/>
+	</link>
+	<link name="gripper_b">
+		<visual>
+			<origin rpy="0 0 0" xyz="0 0 0"/>
+			<geometry>
+				<mesh filename="package://mover6_description/meshes/gripper_b.STL"  scale="1 1 1"/>
+			</geometry>
+		</visual>
+		<collision>
+			<origin xyz="0 0 0" rpy="0 0 0" />
+			<geometry>
+				<mesh filename="package://mover6_description/meshes/gripper_b.STL" scale="1 1 1"/>
+			</geometry>
+		</collision>
+		<xacro:default_inertial z_value="0" mass="0.1"/>
+	</link>
 	<joint name="joint1" type="revolute">
 		<axis xyz="0 0 -1"/>
@@ -173,4 +218,28 @@
 		<joint_properties damping="1.0" friction="1.0"/>
 	</joint>
+	<joint name="joint7" type="fixed">
+		<axis xyz="0 0 1"/>
+		<parent link="link6"/>
+		<child link="link7"/>
+		<origin rpy="3.14159 0 1.5708" xyz="0 0 0"/>
+		<limit lower="-2.09" upper="2.09" effort="100" velocity="100"/>
+		<joint_properties damping="1.0" friction="1.0"/>
+	</joint>
+	<joint name="joint_gripper_a" type="revolute">
+		<axis xyz="0 0 1"/>
+		<parent link="link7"/>
+		<child link="gripper_a"/>
+		<origin rpy="1.5708 -0.33752 3.1416" xyz="-0.0055607 -0.0041434 -0.04688"/>
+		<limit lower="-1" upper="1" effort="100" velocity="100"/>
+		<joint_properties damping="1.0" friction="1.0"/>
+	</joint>
+	<joint name="joint_gripper_b" type="revolute">
+		<axis xyz="0 0 1"/>
+		<parent link="link7"/>
+		<child link="gripper_b"/>
+		<origin rpy="1.5708 -0.33752 0" xyz="0.0055607 0.005 -0.04688"/>
+		<limit lower="-1" upper="1" effort="100" velocity="100"/>
+		<joint_properties damping="1.0" friction="1.0"/>
+	</joint>
 	<transmission name="tran1">
 		<type>transmission_interface/SimpleTransmission</type>
@@ -229,4 +298,24 @@
 		</joint>
 		<actuator name="motor6">
+		    <hardwareInterface>hardware_interface/EffortJointInterface</hardwareInterface>
+			<mechanicalReduction>1</mechanicalReduction>
+		</actuator>
+	</transmission>
+	<transmission name="tran7">
+		<type>transmission_interface/SimpleTransmission</type>
+		<joint name="joint_gripper_a">
+			<hardwareInterface>hardware_interface/EffortJointInterface</hardwareInterface>
+		</joint>
+		<actuator name="motor7">
+		    <hardwareInterface>hardware_interface/EffortJointInterface</hardwareInterface>
+			<mechanicalReduction>1</mechanicalReduction>
+		</actuator>
+	</transmission>
+	<transmission name="tran8">
+		<type>transmission_interface/SimpleTransmission</type>
+		<joint name="joint_gripper_b">
+			<hardwareInterface>hardware_interface/EffortJointInterface</hardwareInterface>
+		</joint>
+		<actuator name="gripper_b">
 		    <hardwareInterface>hardware_interface/EffortJointInterface</hardwareInterface>
 			<mechanicalReduction>1</mechanicalReduction>

Commit message: trying new values for all then updating to be better

File: src/mover6_description/urdf/CPRMover6.urdf.xacro (robot description, xacro)
@@ -174,6 +174,6 @@
 		<child link="link1"/>
 		<origin rpy="0 0 0" xyz="0 0 0.130"/>
-		<limit lower="-2.27" upper="2.27" effort="100" velocity="30"/>
-		<joint_properties damping="1.0" friction="10.0"/>
+		<limit lower="-2.27" upper="2.27" effort="10" velocity="0.15"/>
+		<joint_properties damping="10.0" friction="100.0"/>
 	</joint>
 	<joint name="joint2" type="revolute">
@@ -182,6 +182,6 @@
 		<child link="link2"/>
 		<origin rpy="0 0 0" xyz="0 0 0.0625"/>
-		<limit lower="-0.87" upper="1.05" effort="100" velocity="30"/>
-		<joint_properties damping="1.0" friction="10.0"/>
+		<limit lower="-0.87" upper="1.05" effort="1000000" velocity="0.0015"/>
+		<joint_properties damping="10.0" friction="10000.0"/>
 	</joint>
 	<joint name="joint3" type="revolute">
@@ -190,6 +190,6 @@
 		<child link="link3"/>
 		<origin rpy="0 1.57079632679 0" xyz="0 0 0.190"/>
-		<limit lower="-1.92" upper="1.31" effort="100" velocity="30"/>
-		<joint_properties damping="1.0" friction="10.0"/>
+		<limit lower="-1.92" upper="1.31" effort="10" velocity="0.15"/>
+		<joint_properties damping="10.0" friction="100.0"/>
 	</joint>
 	<joint name="joint4" type="revolute">
@@ -198,6 +198,6 @@
 		<child link="link4"/>
 		<origin rpy="0 0 0" xyz="-0.06 0 0"/>
-		<limit lower="-2.44" upper="2.44" effort="100" velocity="30"/>
-		<joint_properties damping="1.0" friction="10.0"/>
+		<limit lower="-2.44" upper="2.44" effort="10" velocity="0.15"/>
+		<joint_properties damping="10.0" friction="100.0"/>
 	</joint>
 	<joint name="joint5" type="revolute">

Commit message: values getting better

File: src/mover6_description/urdf/CPRMover6.urdf.xacro (robot description, xacro)
@@ -182,6 +182,6 @@
 		<child link="link2"/>
 		<origin rpy="0 0 0" xyz="0 0 0.0625"/>
-		<limit lower="-0.87" upper="1.05" effort="1000000" velocity="0.0015"/>
-		<joint_properties damping="10.0" friction="10000.0"/>
+		<limit lower="-0.87" upper="1.05" effort="100" velocity="0.0015"/>
+		<joint_properties damping="10000.0" friction="10000000.0"/>
 	</joint>
 	<joint name="joint3" type="revolute">

Commit message: not good valies

File: src/mover6_description/urdf/CPRMover6.urdf.xacro (robot description, xacro)
@@ -182,6 +182,6 @@
 		<child link="link2"/>
 		<origin rpy="0 0 0" xyz="0 0 0.0625"/>
-		<limit lower="-0.87" upper="1.05" effort="100" velocity="0.0015"/>
-		<joint_properties damping="10000.0" friction="10000000.0"/>
+		<limit lower="-0.87" upper="1.05" effort="1000" velocity="0.0015"/>
+		<joint_properties damping="1000.0" friction="100000.0"/>
 	</joint>
 	<joint name="joint3" type="revolute">

Commit message: removing mass

File: src/mover6_description/urdf/CPRMover6.urdf.xacro (robot description, xacro)
@@ -19,4 +19,14 @@
 		</inertial>
 	</xacro:macro>
+		<!-- Joint 2 Inertial -->
+	<xacro:macro name="j2_inertial" params="z_value mass">
+		<inertial>
+			<origin xyz="0 0 ${z_value}" rpy="0 0 0"/>
+			<mass value="${mass}" />
+			<inertia ixx="0.001" ixy="0.0" ixz="0.0"
+               iyy="0.001" iyz="0.0"
+               izz="0.001" />
+		</inertial>
+	</xacro:macro>
 	<link name="base_link">
 		<visual>
@@ -47,5 +57,5 @@
 			</geometry>
 		</collision>
-		<xacro:default_inertial z_value="0" mass="0.5"/>
+		<xacro:j2_inertial z_value="0" mass="0.0"/>
 	</link>
 	<link name="link2">
@@ -62,5 +72,5 @@
 			</geometry>
 		</collision>
-		<xacro:default_inertial z_value="0" mass="0.5"/>
+		<xacro:default_inertial z_value="0" mass="0.0"/>
 	</link>
 	<link name="link3">
@@ -77,5 +87,5 @@
 			</geometry>
 		</collision>
-		<xacro:default_inertial z_value="0" mass="0.5"/>
+		<xacro:default_inertial z_value="0" mass="0.0"/>
 	</link>
 	<link name="link4">
@@ -92,5 +102,5 @@
 			</geometry>
 		</collision>
-		<xacro:default_inertial z_value="0" mass="0.2"/>
+		<xacro:default_inertial z_value="0" mass="0.0"/>
 	</link>
 	<link name="link5">
@@ -107,5 +117,5 @@
 			</geometry>
 		</collision>
-		<xacro:default_inertial z_value="0" mass="0.2"/>
+		<xacro:default_inertial z_value="0" mass="0.0"/>
 	</link>
 	<link name="link6">
@@ -137,5 +147,5 @@
 			</geometry>
 		</collision>
-		<xacro:default_inertial z_value="0" mass="0.1"/>
+		<xacro:default_inertial z_value="0" mass="0.0"/>
 	</link>
 	<link name="gripper_a">
@@ -152,5 +162,5 @@
 			</geometry>
 		</collision>
-		<xacro:default_inertial z_value="0" mass="0.1"/>
+		<xacro:default_inertial z_value="0" mass="0.0"/>
 	</link>
 	<link name="gripper_b">
@@ -167,5 +177,5 @@
 			</geometry>
 		</collision>
-		<xacro:default_inertial z_value="0" mass="0.1"/>
+		<xacro:default_inertial z_value="0" mass="0.0"/>
 	</link>
 	<joint name="joint1" type="revolute">
@@ -182,6 +192,6 @@
 		<child link="link2"/>
 		<origin rpy="0 0 0" xyz="0 0 0.0625"/>
-		<limit lower="-0.87" upper="1.05" effort="1000" velocity="0.0015"/>
-		<joint_properties damping="1000.0" friction="100000.0"/>
+		<limit lower="-0.87" upper="1.05" effort="1000" velocity="0.15"/>
+		<joint_properties damping="10000.0" friction="100.0"/>
 	</joint>
 	<joint name="joint3" type="revolute">
