Commit message: final values for tonight poroibably

File: src/mover6_description/urdf/CPRMover6.urdf.xacro (robot description, xacro)
@@ -24,7 +24,7 @@
 			<origin xyz="0 0 ${z_value}" rpy="0 0 0"/>
 			<mass value="${mass}" />
-			<inertia ixx="0.001" ixy="0.0" ixz="0.0"
-               iyy="0.001" iyz="0.0"
-               izz="0.001" />
+			<inertia ixx="0.01" ixy="0.0" ixz="0.0"
+               iyy="0.01" iyz="0.0"
+               izz="0.01" />
 		</inertial>
 	</xacro:macro>
@@ -57,5 +57,5 @@
 			</geometry>
 		</collision>
-		<xacro:j2_inertial z_value="0" mass="0.0001"/>
+		<xacro:j2_inertial z_value="0" mass="0.01"/>
 	</link>
 	<link name="link2">
@@ -72,5 +72,5 @@
 			</geometry>
 		</collision>
-		<xacro:default_inertial z_value="0" mass="0.0001"/>
+		<xacro:default_inertial z_value="0" mass="0.01"/>
 	</link>
 	<link name="link3">
@@ -87,5 +87,5 @@
 			</geometry>
 		</collision>
-		<xacro:default_inertial z_value="0" mass="0.0001"/>
+		<xacro:default_inertial z_value="0" mass="0.01"/>
 	</link>
 	<link name="link4">
@@ -102,5 +102,5 @@
 			</geometry>
 		</collision>
-		<xacro:default_inertial z_value="0" mass="0.0001"/>
+		<xacro:default_inertial z_value="0" mass="0.01"/>
 	</link>
 	<link name="link5">
@@ -117,5 +117,5 @@
 			</geometry>
 		</collision>
-		<xacro:default_inertial z_value="0" mass="0.0001"/>
+		<xacro:default_inertial z_value="0" mass="0.01"/>
 	</link>
 	<link name="link6">
@@ -132,5 +132,5 @@
 			</geometry>
 		</collision>
-		<xacro:default_inertial z_value="0" mass="0.0001"/>
+		<xacro:default_inertial z_value="0" mass="0.01"/>
 	</link>
 	<link name="link7">
@@ -147,5 +147,5 @@
 			</geometry>
 		</collision>
-		<xacro:default_inertial z_value="0" mass="0.0001"/>
+		<xacro:default_inertial z_value="0" mass="0.01"/>
 	</link>
 	<link name="gripper_a">
@@ -162,5 +162,5 @@
 			</geometry>
 		</collision>
-		<xacro:default_inertial z_value="0" mass="0.0001"/>
+		<xacro:default_inertial z_value="0" mass="0.01"/>
 	</link>
 	<link name="gripper_b">
@@ -177,5 +177,5 @@
 			</geometry>
 		</collision>
-		<xacro:default_inertial z_value="0" mass="0.0001"/>
+		<xacro:default_inertial z_value="0" mass="0.01"/>
 	</link>
 	<joint name="joint1" type="revolute">

Commit message: joint 3 conreoll

File: src/mover6_description/urdf/CPRMover6.urdf.xacro (robot description, xacro)
@@ -24,7 +24,7 @@
 			<origin xyz="0 0 ${z_value}" rpy="0 0 0"/>
 			<mass value="${mass}" />
-			<inertia ixx="0.01" ixy="0.0" ixz="0.0"
-               iyy="0.01" iyz="0.0"
-               izz="0.01" />
+			<inertia ixx="1" ixy="0.0" ixz="0.0"
+               iyy="1" iyz="0.0"
+               izz="1" />
 		</inertial>
 	</xacro:macro>
@@ -117,5 +117,5 @@
 			</geometry>
 		</collision>
-		<xacro:default_inertial z_value="0" mass="0.01"/>
+		<xacro:default_inertial z_value="0" mass="0.1"/>
 	</link>
 	<link name="link6">
@@ -132,5 +132,5 @@
 			</geometry>
 		</collision>
-		<xacro:default_inertial z_value="0" mass="0.01"/>
+		<xacro:default_inertial z_value="0" mass="0.1"/>
 	</link>
 	<link name="link7">
@@ -147,5 +147,5 @@
 			</geometry>
 		</collision>
-		<xacro:default_inertial z_value="0" mass="0.01"/>
+		<xacro:default_inertial z_value="0" mass="0.1"/>
 	</link>
 	<link name="gripper_a">
@@ -162,5 +162,5 @@
 			</geometry>
 		</collision>
-		<xacro:default_inertial z_value="0" mass="0.01"/>
+		<xacro:default_inertial z_value="0" mass="0.1"/>
 	</link>
 	<link name="gripper_b">
@@ -192,6 +192,6 @@
 		<child link="link2"/>
 		<origin rpy="0 0 0" xyz="0 0 0.0625"/>
-		<limit lower="-0.87" upper="1.05" effort="1000" velocity="0.15"/>
-		<joint_properties damping="10000.0" friction="100.0"/>
+		<limit lower="-0.87" upper="1.05" effort="100" velocity="0.01"/>
+		<joint_properties damping="100.0" friction="100.0"/>
 	</joint>
 	<joint name="joint3" type="revolute">
@@ -201,5 +201,5 @@
 		<origin rpy="0 1.57079632679 0" xyz="0 0 0.190"/>
 		<limit lower="-1.92" upper="1.31" effort="10" velocity="0.15"/>
-		<joint_properties damping="10.0" friction="100.0"/>
+		<joint_properties damping="100.0" friction="10000.0"/>
 	</joint>
 	<joint name="joint4" type="revolute">

Commit message: incressing the gain

File: src/mover6_description/urdf/CPRMover6.urdf.xacro (robot description, xacro)
@@ -200,6 +200,6 @@
 		<child link="link3"/>
 		<origin rpy="0 1.57079632679 0" xyz="0 0 0.190"/>
-		<limit lower="-1.92" upper="1.31" effort="10" velocity="0.15"/>
-		<joint_properties damping="100.0" friction="10000.0"/>
+		<limit lower="-1.92" upper="1.31" effort="10" velocity="0.05"/>
+		<joint_properties damping="100.0" friction="1000.0"/>
 	</joint>
 	<joint name="joint4" type="revolute">

Commit message: less effort

File: src/mover6_description/urdf/CPRMover6.urdf.xacro (robot description, xacro)
@@ -200,6 +200,6 @@
 		<child link="link3"/>
 		<origin rpy="0 1.57079632679 0" xyz="0 0 0.190"/>
-		<limit lower="-1.92" upper="1.31" effort="10" velocity="0.05"/>
-		<joint_properties damping="100.0" friction="1000.0"/>
+		<limit lower="-1.92" upper="1.31" effort="1" velocity="0.05"/>
+		<joint_properties damping="10000.0" friction="1000.0"/>
 	</joint>
 	<joint name="joint4" type="revolute">

Commit message: hopefully finbal valeus]

File: src/mover6_description/urdf/CPRMover6.urdf.xacro (robot description, xacro)
@@ -185,5 +185,5 @@
 		<origin rpy="0 0 0" xyz="0 0 0.130"/>
 		<limit lower="-2.27" upper="2.27" effort="10" velocity="0.15"/>
-		<joint_properties damping="10.0" friction="100.0"/>
+		<joint_properties damping="20.0" friction="120.0"/>
 	</joint>
 	<joint name="joint2" type="revolute">
@@ -192,6 +192,6 @@
 		<child link="link2"/>
 		<origin rpy="0 0 0" xyz="0 0 0.0625"/>
-		<limit lower="-0.87" upper="1.05" effort="100" velocity="0.01"/>
-		<joint_properties damping="100.0" friction="100.0"/>
+		<limit lower="-0.87" upper="1.05" effort="10" velocity="0.15"/>
+		<joint_properties damping="10.0" friction="150.0"/>
 	</joint>
 	<joint name="joint3" type="revolute">
@@ -200,6 +200,6 @@
 		<child link="link3"/>
 		<origin rpy="0 1.57079632679 0" xyz="0 0 0.190"/>
-		<limit lower="-1.92" upper="1.31" effort="1" velocity="0.05"/>
-		<joint_properties damping="10000.0" friction="1000.0"/>
+		<limit lower="-1.92" upper="1.31" effort="10" velocity="0.15"/>
+		<joint_properties damping="10.0" friction="100.0"/>
 	</joint>
 	<joint name="joint4" type="revolute">
@@ -216,6 +216,6 @@
 		<child link="link5"/>
 		<origin rpy="0 0 0" xyz="0 0 0.290"/>
-		<limit lower="-1.22" upper="1.05" effort="100" velocity="40"/>
-		<joint_properties damping="1.0" friction="1.0"/>
+		<limit lower="-1.22" upper="1.05" effort="10" velocity="0.15"/>
+		<joint_properties damping="10.0" friction="100.0"/>
 	</joint>
 	<joint name="joint6" type="revolute">
@@ -224,6 +224,6 @@
 		<child link="link6"/>
 		<origin rpy="0 0 0" xyz="0 0 0.055"/>
-		<limit lower="-2.09" upper="2.09" effort="100" velocity="100"/>
-		<joint_properties damping="1.0" friction="1.0"/>
+		<limit lower="-2.09" upper="2.09" effort="10" velocity="0.15"/>
+		<joint_properties damping="10.0" friction="100.0"/>
 	</joint>
 	<joint name="joint7" type="fixed">
@@ -232,6 +232,6 @@
 		<child link="link7"/>
 		<origin rpy="3.14159 0 1.5708" xyz="0 0 0"/>
-		<limit lower="-2.09" upper="2.09" effort="100" velocity="100"/>
-		<joint_properties damping="1.0" friction="1.0"/>
+		<limit lower="-2.09" upper="2.09" effort="10" velocity="0.15"/>
+		<joint_properties damping="10.0" friction="100.0"/>
 	</joint>
 	<joint name="joint_gripper_a" type="revolute">
@@ -335,3 +335,30 @@
     </plugin>
     </gazebo>
+	<gazebo reference="link1">
+		<gravity>0</gravity>
+	</gazebo>
+	<gazebo reference="link2">
+		<gravity>0</gravity>
+	</gazebo>
+	<gazebo reference="link3">
+		<gravity>0</gravity>
+	</gazebo>
+	<gazebo reference="link4">
+		<gravity>0</gravity>
+	</gazebo>
+	<gazebo reference="link5">
+		<gravity>0</gravity>
+	</gazebo>
+	<gazebo reference="link6">
+		<gravity>0</gravity>
+	</gazebo>
+	<gazebo reference="link7">
+		<gravity>0</gravity>
+	</gazebo>
+	<gazebo reference="gripper_a">
+		<gravity>0</gravity>
+	</gazebo>
+	<gazebo reference="gripper_b">
+		<gravity>0</gravity>
+	</gazebo>
 </robot>

Commit message: final values and plots

File: src/mover6_description/urdf/CPRMover6.urdf.xacro (robot description, xacro)
@@ -200,5 +200,5 @@
 		<child link="link3"/>
 		<origin rpy="0 1.57079632679 0" xyz="0 0 0.190"/>
-		<limit lower="-1.92" upper="1.31" effort="10" velocity="0.15"/>
+		<limit lower="-1.92" upper="1.31" effort="10" velocity="0.1"/>
 		<joint_properties damping="10.0" friction="100.0"/>
 	</joint>
@@ -208,5 +208,5 @@
 		<child link="link4"/>
 		<origin rpy="0 0 0" xyz="-0.06 0 0"/>
-		<limit lower="-2.44" upper="2.44" effort="10" velocity="0.15"/>
+		<limit lower="-2.44" upper="2.44" effort="10" velocity="0.06"/>
 		<joint_properties damping="10.0" friction="100.0"/>
 	</joint>
@@ -216,5 +216,5 @@
 		<child link="link5"/>
 		<origin rpy="0 0 0" xyz="0 0 0.290"/>
-		<limit lower="-1.22" upper="1.05" effort="10" velocity="0.15"/>
+		<limit lower="-1.22" upper="1.05" effort="10" velocity="0.03"/>
 		<joint_properties damping="10.0" friction="100.0"/>
 	</joint>
@@ -224,5 +224,5 @@
 		<child link="link6"/>
 		<origin rpy="0 0 0" xyz="0 0 0.055"/>
-		<limit lower="-2.09" upper="2.09" effort="10" velocity="0.15"/>
+		<limit lower="-2.09" upper="2.09" effort="10" velocity="0.03"/>
 		<joint_properties damping="10.0" friction="100.0"/>
 	</joint>

Commit message: Fixing Simulation Robot Behaviour (#62)
* Tweak joint5 pid parameters

* UPDING TO INCUDE THE PHOCAL

* splitting the bad veriable

* changing speed of phoical

* undo

* trying new values for all then updating to be better

* values getting better

* not good valies

* removing mass

* small joints mass

* dont spawn inside eachother

* final values for tonight poroibably

* cakin make much was bad

* joint 3 conreoll

* incressing the gain

* pid correct

* less effort

* hopefully finbal valeus]

* final values and plots

* Remove imgs

* Set robot distance

* Copy a config to b

---------

Co-authored-by: tomrrr <tomtommrichards@gmail.com>

File: src/mover6_description/urdf/CPRMover6.urdf.xacro (robot description, xacro)
@@ -19,4 +19,14 @@
 		</inertial>
 	</xacro:macro>
+		<!-- Joint 2 Inertial -->
+	<xacro:macro name="j2_inertial" params="z_value mass">
+		<inertial>
+			<origin xyz="0 0 ${z_value}" rpy="0 0 0"/>
+			<mass value="${mass}" />
+			<inertia ixx="1" ixy="0.0" ixz="0.0"
+               iyy="1" iyz="0.0"
+               izz="1" />
+		</inertial>
+	</xacro:macro>
 	<link name="base_link">
 		<visual>
@@ -47,5 +57,5 @@
 			</geometry>
 		</collision>
-		<xacro:default_inertial z_value="0" mass="0.5"/>
+		<xacro:j2_inertial z_value="0" mass="0.01"/>
 	</link>
 	<link name="link2">
@@ -62,5 +72,5 @@
 			</geometry>
 		</collision>
-		<xacro:default_inertial z_value="0" mass="0.5"/>
+		<xacro:default_inertial z_value="0" mass="0.01"/>
 	</link>
 	<link name="link3">
@@ -77,5 +87,5 @@
 			</geometry>
 		</collision>
-		<xacro:default_inertial z_value="0" mass="0.5"/>
+		<xacro:default_inertial z_value="0" mass="0.01"/>
 	</link>
 	<link name="link4">
@@ -92,5 +102,5 @@
 			</geometry>
 		</collision>
-		<xacro:default_inertial z_value="0" mass="0.2"/>
+		<xacro:default_inertial z_value="0" mass="0.01"/>
 	</link>
 	<link name="link5">
@@ -107,5 +117,5 @@
 			</geometry>
 		</collision>
-		<xacro:default_inertial z_value="0" mass="0.2"/>
+		<xacro:default_inertial z_value="0" mass="0.1"/>
 	</link>
 	<link name="link6">
@@ -167,5 +177,5 @@
 			</geometry>
 		</collision>
-		<xacro:default_inertial z_value="0" mass="0.1"/>
+		<xacro:default_inertial z_value="0" mass="0.01"/>
 	</link>
 	<joint name="joint1" type="revolute">
@@ -174,6 +184,6 @@
 		<child link="link1"/>
 		<origin rpy="0 0 0" xyz="0 0 0.130"/>
-		<limit lower="-2.27" upper="2.27" effort="100" velocity="30"/>
-		<joint_properties damping="1.0" friction="10.0"/>
+		<limit lower="-2.27" upper="2.27" effort="10" velocity="0.15"/>
+		<joint_properties damping="20.0" friction="120.0"/>
 	</joint>
 	<joint name="joint2" type="revolute">
@@ -182,6 +192,6 @@
 		<child link="link2"/>
 		<origin rpy="0 0 0" xyz="0 0 0.0625"/>
-		<limit lower="-0.87" upper="1.05" effort="100" velocity="30"/>
-		<joint_properties damping="1.0" friction="10.0"/>
+		<limit lower="-0.87" upper="1.05" effort="10" velocity="0.15"/>
+		<joint_properties damping="10.0" friction="150.0"/>
 	</joint>
 	<joint name="joint3" type="revolute">
@@ -190,6 +200,6 @@
 		<child link="link3"/>
 		<origin rpy="0 1.57079632679 0" xyz="0 0 0.190"/>
-		<limit lower="-1.92" upper="1.31" effort="100" velocity="30"/>
-		<joint_properties damping="1.0" friction="10.0"/>
+		<limit lower="-1.92" upper="1.31" effort="10" velocity="0.1"/>
+		<joint_properties damping="10.0" friction="100.0"/>
 	</joint>
 	<joint name="joint4" type="revolute">
@@ -198,6 +208,6 @@
 		<child link="link4"/>
 		<origin rpy="0 0 0" xyz="-0.06 0 0"/>
-		<limit lower="-2.44" upper="2.44" effort="100" velocity="30"/>
-		<joint_properties damping="1.0" friction="10.0"/>
+		<limit lower="-2.44" upper="2.44" effort="10" velocity="0.06"/>
+		<joint_properties damping="10.0" friction="100.0"/>
 	</joint>
 	<joint name="joint5" type="revolute">
@@ -206,6 +216,6 @@
 		<child link="link5"/>
 		<origin rpy="0 0 0" xyz="0 0 0.290"/>
-		<limit lower="-1.22" upper="1.05" effort="100" velocity="40"/>
-		<joint_properties damping="1.0" friction="1.0"/>
+		<limit lower="-1.22" upper="1.05" effort="10" velocity="0.03"/>
+		<joint_properties damping="10.0" friction="100.0"/>
 	</joint>
 	<joint name="joint6" type="revolute">
@@ -214,6 +224,6 @@
 		<child link="link6"/>
 		<origin rpy="0 0 0" xyz="0 0 0.055"/>
-		<limit lower="-2.09" upper="2.09" effort="100" velocity="100"/>
-		<joint_properties damping="1.0" friction="1.0"/>
+		<limit lower="-2.09" upper="2.09" effort="10" velocity="0.03"/>
+		<joint_properties damping="10.0" friction="100.0"/>
 	</joint>
 	<joint name="joint7" type="fixed">
@@ -222,6 +232,6 @@
 		<child link="link7"/>
 		<origin rpy="3.14159 0 1.5708" xyz="0 0 0"/>
-		<limit lower="-2.09" upper="2.09" effort="100" velocity="100"/>
-		<joint_properties damping="1.0" friction="1.0"/>
+		<limit lower="-2.09" upper="2.09" effort="10" velocity="0.15"/>
+		<joint_properties damping="10.0" friction="100.0"/>
 	</joint>
 	<joint name="joint_gripper_a" type="revolute">
@@ -325,3 +335,30 @@
     </plugin>
     </gazebo>
+	<gazebo reference="link1">
+		<gravity>0</gravity>
+	</gazebo>
+	<gazebo reference="link2">
+		<gravity>0</gravity>
+	</gazebo>
+	<gazebo reference="link3">
+		<gravity>0</gravity>
+	</gazebo>
+	<gazebo reference="link4">
+		<gravity>0</gravity>
+	</gazebo>
+	<gazebo reference="link5">
+		<gravity>0</gravity>
+	</gazebo>
+	<gazebo reference="link6">
+		<gravity>0</gravity>
+	</gazebo>
+	<gazebo reference="link7">
+		<gravity>0</gravity>
+	</gazebo>
+	<gazebo reference="gripper_a">
+		<gravity>0</gravity>
+	</gazebo>
+	<gazebo reference="gripper_b">
+		<gravity>0</gravity>
+	</gazebo>
 </robot>
