Commit message: Fix block size

File: src/block_controller/urdf/block.urdf (robot description, URDF)
Before this commit: robot block, 1 links, 0 joints
Links:
- link box: mass 1.0 -> 0.2; geometry collision box size=0.1 0.02 0.02; visual box size=0.1 0.02 0.02

Commit message: Finalised random block spawner

File: src/block_controller/urdf/block.urdf (robot description, URDF)
Before this commit: robot block, 1 links, 0 joints
Links:
- link box: mass 0.2 -> 0.02; geometry collision box size=0.06 0.02 0.01; visual box size=0.06 0.02 0.01

Commit message: Edit block urdf

File: src/block_controller/urdf/block.urdf (robot description, URDF)
Before this commit: robot block, 1 links, 0 joints
Links:
- link box: mass 0.02 -> 0.2

Commit message: tf experimenting

File: src/block_controller/urdf/block.urdf (robot description, URDF)
Before this commit: robot block, 1 links, 0 joints
Links:
- link box: geometry collision box size=0.105 0.035 0.035; visual box size=0.105 0.035 0.035
